File: analog_frontend.kicad_sch (KiCad schematic)
At the start: 38 parts

Commit message: Update: slowly drawing schematic
Parts:
- removed C? (x5): C, symbol Device:C
- removed C? (x2): 1n, symbol Device:C
- removed C? (x2): 1u, symbol Device:C
- removed C? (x2): 510p, symbol Device:C
- removed C?: 10n, symbol Device:C
- removed D? (x4): BAT54, symbol Device:D_Schottky
- removed D? (x2): 1N4148, symbol Device:D
- removed J? (x2): IN1, symbol Connector:Conn_Coaxial
- removed L? (x4): L, symbol Device:L
- removed R? (x2): 0, symbol Device:R
- removed R? (x6): 100, symbol Device:R
- removed R?: 10k, symbol Device:R
- removed R? (x2): R, symbol Device:R
- removed R?: 50, symbol Device:R
- removed U?: THS4521ID, Package_SO:SOIC-8_3.9x4.9mm_P1.27mm, symbol symbols:THS4521ID
- removed U?: AD7357xRU, Package_SO:TSSOP-16_4.4x5mm_P0.65mm, symbol symbols:AD7357xRU
Other:
- removed sheet Input Amplifier 1
- removed sheet Input Amplifier1
