File: lwdo-sdr.kicad_sch (KiCad schematic)
At the start: 0 parts

Commit message: Update: slowly drawing schematic
Parts:
- added C101, C102: 27p, symbol Device:C
- added C103, C104, C105, C106: 10u 6.3v, symbol Device:C_Polarized
- added C107, C108, C109, C110, C114, C115, C116, C? (x8): 100n, symbol Device:C
- added C111: 10n, symbol Device:C
- added C112, C113, C?: 4.7u, symbol Device:C
- added C117: 10u, symbol Device:C
- added C?: 22u 16V, symbol Device:C_Polarized
- added C?: 1u, symbol Device:C
- added D101: PESD2USB3U, symbol Device:D_Zener_Dual_CommonAnode_KKA_Parallel
- added D102: D_Zener, symbol Device:D_Zener
- added D103, D104, D105, D106: SBR3U40S1F, symbol Device:D_Schottky
- added D?: BAT54J, Diode_SMD:D_SOD-323F, symbol Diode:BAT54J
- added FB101, FB102, FB103: FerriteBead, symbol Device:FerriteBead
- added J101: IN1, symbol Connector:Conn_Coaxial
- added J102: IN2, symbol Connector:Conn_Coaxial
- added J103: IN3, symbol Connector:Conn_Coaxial
- added J104: IN4, symbol Connector:Conn_Coaxial
- added J105: USB_B, Connector_USB:USB_B_Lumberg_2411_02_Horizontal, symbol Connector:USB_B
- added JP?: SUSP_MODE, symbol Jumper:Jumper_3_Bridged12
- added Q101: DMP2120U, symbol Device:Q_PMOS_GSD
- added Q? (x2): 2N7002, Package_TO_SOT_SMD:SOT-23, symbol Transistor_FET:2N7002
- added R101, R102, R104, R108, R109, R111: 10k, symbol Device:R
- added R103: 2.2k, symbol Device:R
- added R105, R107: 0, symbol Device:R
- added R106: 12k, symbol Device:R
- added R110: 5.1k, symbol Device:R
- added R?: 0.047, symbol Device:R
- added R?: 4.7k, symbol Device:R
- added R?: 100k, symbol Device:R
- added U101: AT93C56, symbol Memory_EEPROM:93CxxC
- added U102: FT2232HL, Package_QFP:LQFP-64_10x10mm_P0.5mm, symbol Interface_USB:FT2232HL
- added U103, U104: AD7357xRU, Package_SO:TSSOP-16_4.4x5mm_P0.65mm, symbol symbols:AD7357xRU
- added U105: ICE40HX4K, Package_QFP:TQFP-144_20x20mm_P0.5mm, symbol FPGA_Lattice:ICE40HX4K-TQ144
- added U?: NCP1117-3.3, Package_TO_SOT_SMD:SOT-223-3_TabPin2, symbol Regulator_Linear:NCP1117-3.3_SOT223
- added Y101: 12MHz, symbol Device:Crystal_GND24
Connections:
- new net: R103.1, U101.3 (DI), U102.61 (EEDATA)
- new net: R101.1, R103.2, U101.4 (DO)
- new net: C?.1, D105.1 (K), D106.1 (K), U?.3 (VI)
- new net: D101.2 (K), J105.2 (D-), R105.1
- new net: D101.1 (K), J105.3 (D+), R107.1
- new net: R?.2, U?.2 (VO)
- new net: C104.1, C108.1, U103.6 (REFB)
- new net: C106.1, C110.1, U104.6 (REFB)
- new net: U105.30 (VCCIO_3), U105.6 (VCCIO_3)
- new net: D?.1 (K), Q?.3 (D)
- new net: D?.2 (A), JP?.2 (C), R?.2
- new net: R107.2, U102.8 (DP)
- new net: U105.46 (VCCIO_2), U105.57 (VCCIO_2)
- new net: C103.1, C107.1, U103.3 (REFA)
- new net: C?.2, Q101.1 (G), R?.1, R?.2
- new net: R105.2, U102.7 (DM)
- new net: JP?.1 (A), Q?.3 (D)
- new net: R108.2, U102.14 (~{RESET})
- new net: C101.1, U102.2 (OSCI), Y101.1
- new net: C102.1, U102.3 (OSCO), Y101.3
- new net: R109.1, U102.53 (BCBUS2)
- new net: R106.1, U102.6 (REF)
- new net: R102.1, U101.2 (SCLK), U102.62 (EECLK)
- new net: R104.1, U101.1 (CS), U102.63 (EECS)
- new net: C105.1, C109.1, U104.3 (REFA)
- new net: U105.123 (VCCIO_0), U105.131 (VCCIO_0)
- new net: U105.100 (VCCIO_1), U105.89 (VCCIO_1)
- new net: U105.111 (VCC), U105.27 (VCC), U105.40 (VCC), U105.92 (VCC)
- new net +2V5A: U103.9 (VDD), U104.9 (VDD)
- new net +3V3D: U103.16 (VDRIVE), U104.16 (VDRIVE)
- new net +5VEXT: D103.2 (A), D105.2 (A)
- new net +5VMAIN: D103.1 (K), D104.1 (K)
- new net AGND: C103.2, C104.2, C105.2, C106.2, C107.2, C108.2, C109.2, C110.2, J101.2 (Ext), J102.2 (Ext), J103.2 (Ext), J104.2 (Ext), U103.11 (AGND), U103.4 (REFGND), U103.5 (AGND), U104.11 (AGND), U104.4 (REFGND), U104.5 (AGND)
- new net FT_+1V8: C?.1, C?.1, C?.1, C?.1, U102.12 (VCORE), U102.37 (VCORE), U102.49 (VREGOUT), U102.64 (VCORE)
- new net FT_+3V3: C?.1, C?.1, C?.1, C?.1, C?.1, FB101.2, FB102.2, Q?.1 (G), R101.2, R102.2, R104.2, R108.1, R109.2, R?.1, U101.6 (ORG), U101.8 (VCC), U102.20 (VCCIO), U102.31 (VCCIO), U102.42 (VCCIO), U102.50 (VREGIN), U102.56 (VCCIO)
- new net FT_CDONE: U102.44 (BDBUS5)
- new net FT_FIFO.CLKOUT: U102.32 (ACBUS5)
- new net FT_FIFO.D0: U102.16 (ADBUS0)
- new net FT_FIFO.D1: U102.17 (ADBUS1)
- new net FT_FIFO.D2: U102.18 (ADBUS2)
- new net FT_FIFO.D3: U102.19 (ADBUS3)
- new net FT_FIFO.D4: U102.21 (ADBUS4)
- new net FT_FIFO.D5: U102.22 (ADBUS5)
- new net FT_FIFO.D6: U102.23 (ADBUS6)
- new net FT_FIFO.D7: U102.24 (ADBUS7)
- new net FT_FIFO.SIWU: U102.30 (ACBUS4)
- new net FT_FIFO.~{OE}: U102.33 (ACBUS6)
- new net FT_FIFO.~{RD}: U102.28 (ACBUS2)
- new net FT_FIFO.~{RXF}: U102.26 (ACBUS0)
- new net FT_FIFO.~{TXE}: U102.27 (ACBUS1)
- new net FT_FIFO.~{WR}: U102.29 (ACBUS3)
- new net FT_IO1: U102.45 (BDBUS6)
- new net FT_IO2: U102.46 (BDBUS7)
- new net FT_SPI.MISO: U102.40 (BDBUS2)
- new net FT_SPI.MOSI: U102.39 (BDBUS1)
- new net FT_SPI.SCK: U102.38 (BDBUS0)
- new net FT_SPI.~{CS}: U102.41 (BDBUS3)
- new net FT_VPHY: C112.1, C114.1, FB101.1, U102.4 (VPHY)
- new net FT_VPLL: C113.1, C115.1, FB102.1, U102.9 (VPLL)
- new net FT_~{CRESET}: U102.43 (BDBUS4)
- new net FT_~{PWREN}: Q?.2 (S), U102.60 (~{PWREN})
- new net FT_~{PWRSAV}: R110.1, R111.2, U102.59 (BCBUS7)
- new net FT_~{SUSP}: Q?.1 (G), U102.36 (~{SUSPEND})
- new net GND: C101.2, C102.2, C111.2, C112.2, C113.2, C114.2, C115.2, C116.2, C117.2, C?.2, C?.2, C?.2, C?.2, C?.2, C?.2, C?.2, C?.2, C?.2, C?.2, D101.3 (A), D102.2 (A), J105.4 (GND), J105.5 (Shield), JP?.3 (B), Q?.2 (S), R106.2, R111.1, U101.5 (GND), U102.1 (GND), U102.10 (AGND), U102.11 (GND), U102.13 (TEST), U102.15 (GND), U102.25 (GND), U102.35 (GND), U102.47 (GND), U102.5 (GND), U102.51 (GND), U105.103 (GND), U105.13 (GND), U105.132 (GND), U105.14 (GND), U105.140 (GND), U105.5 (GND), U105.59 (GND), U105.69 (GND), U105.86 (GND), U?.1 (GND), Y101.2, Y101.4
- new net GNDD: U103.12 (DGND), U104.12 (DGND)
- new net Input Amplifier 1/IN: J101.1 (In)
- new net Input Amplifier 1/OUT+: U103.2 (INA-)
- new net Input Amplifier 1/OUT-: U103.1 (INA+)
- new net Input Amplifier 2/IN: J102.1 (In)
- new net Input Amplifier 2/OUT+: U103.8 (INB+)
- new net Input Amplifier 2/OUT-: U103.7 (INB-)
- new net Input Amplifier 3/IN: J103.1 (In)
- new net Input Amplifier 3/OUT+: U104.2 (INA-)
- new net Input Amplifier 3/OUT-: U104.1 (INA+)
- new net Input Amplifier 4/IN: J104.1 (In)
- new net Input Amplifier 4/OUT+: U104.8 (INB+)
- new net Input Amplifier 4/OUT-: U104.7 (INB-)
- new net VBUS: C111.1, D102.1 (K), FB103.2, J105.1 (VBUS)
- new net VBUS_CLEAN: C116.1, C117.1, C?.1, D106.2 (A), FB103.1, Q101.2 (S), R110.2, R?.1
- new net VBUS_SWITCHED: D104.2 (A), Q101.3 (D)
Other:
- removed sheet Analog Frontend
- added sheet Input Amplifier 1 (analog_input_amp.kicad_sch)
- added sheet Input Amplifier 2 (analog_input_amp.kicad_sch)
- added sheet Input Amplifier 3 (analog_input_amp.kicad_sch)
- added sheet Input Amplifier 4 (analog_input_amp.kicad_sch)
- note added: "USB inrush current limit: 50uC charge transferred by current _exceeding_ 100mA"

Commit message: Schematic: added VCTCXO, clk out, ref in, separated power supply into a new sheet
Parts:
- removed C104, C105, C106: 10u 6.3v, symbol Device:C_Polarized
- removed C? (x5): 100n, symbol Device:C
- removed C?: 22u 16V, symbol Device:C_Polarized
- removed C?: 1u, symbol Device:C
- removed D103, D104, D105, D106: SBR3U40S1F, symbol Device:D_Schottky
- removed D?: BAT54J, Diode_SMD:D_SOD-323F, symbol Diode:BAT54J
- removed JP?: SUSP_MODE, symbol Jumper:Jumper_3_Bridged12
- removed Q101: DMP2120U, symbol Device:Q_PMOS_GSD
- removed Q? (x2): 2N7002, Package_TO_SOT_SMD:SOT-23, symbol Transistor_FET:2N7002
- removed R?: 0.047, symbol Device:R
- removed R?: 4.7k, symbol Device:R
- removed R?: 100k, symbol Device:R
- removed U?: NCP1117-3.3, Package_TO_SOT_SMD:SOT-223-3_TabPin2, symbol Regulator_Linear:NCP1117-3.3_SOT223
- added C? (x3): 10u/10v, symbol Device:C_Polarized
- added D?: IN1:R,G, LED_THT:LED_D3.0mm-3, symbol Device:LED_Dual_KKA
- added D?: STATUS:R,G, LED_THT:LED_D3.0mm-3, symbol Device:LED_Dual_KKA
- added D?: USB:G, symbol Device:LED
- added D?: IN4:R,G, LED_THT:LED_D3.0mm-3, symbol Device:LED_Dual_KKA
- added D?: IN2:R,G, LED_THT:LED_D3.0mm-3, symbol Device:LED_Dual_KKA
- added D?: IN3:R,G, LED_THT:LED_D3.0mm-3, symbol Device:LED_Dual_KKA
- added J?: REF_IN, symbol Connector:Conn_Coaxial
- added J?: CLK_OUT, symbol Connector:Conn_Coaxial
- added R? (x11): 1k, symbol Device:R
- C103: value 10u 6.3v -> 10u/10v
Connections:
- net VBUS_CLEAN is gone; now on net VBUS: C116.1, C117.1, FB103.1, R110.2
- net +3V3D: now also D?.3 (A), D?.3 (A), D?.3 (A), D?.3 (A), D?.3 (A)
- net AGND: now also C?.2, C?.2, C?.2
- net FT_+3V3: now also D?.2 (A)
- net FT_~{PWREN}: now also R?.2
- net GND: now also J?.2 (Ext), J?.2 (Ext)
- net VBUS: no longer C111.1, D102.1 (K), FB103.2, J105.1 (VBUS)
- net at C108.1, U103.6 (REFB): now also C?.1
- net at C110.1, U104.6 (REFB): now also C?.1
- net at C109.1, U104.3 (REFA): now also C?.1
- new net: C111.1, D102.1 (K), FB103.2, J105.1 (VBUS)
- new net: D?.2 (K2), R?.1 (x5)
- new net: D?.1 (K1), R?.1 (x5)
- new net: D?.1 (K), R?.1
- new net clk_out/OUT: J?.1 (In)
- new net ref_in/IN: J?.1 (In)
- new net ~{LED_IN1G}: R?.2
- new net ~{LED_IN1R}: R?.2
- new net ~{LED_IN2G}: R?.2
- new net ~{LED_IN2R}: R?.2
- new net ~{LED_IN3G}: R?.2
- new net ~{LED_IN3R}: R?.2
- new net ~{LED_IN4G}: R?.2
- new net ~{LED_IN4R}: R?.2
- new net ~{LED_ST_G}: R?.2
- new net ~{LED_ST_R}: R?.2
Other:
- added sheet VCXO (vcxo.kicad_sch)
- added sheet clk_out (clk_out.kicad_sch)
- added sheet power_supply (power_supply.kicad_sch)
- added sheet ref_in (ref_in.kicad_sch)
- moved on the sheet: C111, C116, C117, D102, FB103, J105

Commit message: Schematic updated
Parts:
- removed C101, C102: 27p, symbol Device:C
- removed C111: 10n, symbol Device:C
- removed C113, C?: 4.7u, symbol Device:C
- removed C114, C115, C116, C? (x3): 100n, symbol Device:C
- removed C117: 10u, symbol Device:C
- removed D101: PESD2USB3U, symbol Device:D_Zener_Dual_CommonAnode_KKA_Parallel
- removed D102: D_Zener, symbol Device:D_Zener
- removed FB101, FB102, FB103: FerriteBead, symbol Device:FerriteBead
- removed R101, R102, R104, R109, R111: 10k, symbol Device:R
- removed R103: 2.2k, symbol Device:R
- removed R105: 0, symbol Device:R
- removed R106: 12k, symbol Device:R
- removed R110: 5.1k, symbol Device:R
- removed U101: AT93C56, symbol Memory_EEPROM:93CxxC
- removed U102: FT2232HL, Package_QFP:LQFP-64_10x10mm_P0.5mm, symbol Interface_USB:FT2232HL
- removed Y101: 12MHz, symbol Device:Crystal_GND24
- added C109, C111: 10u, symbol Device:C_Polarized
- added C110: 100n, Capacitor_SMD:C_0805_2012Metric, symbol Device:C
- added JP101: FLASH/CRAM, symbol symbols:Jumper_4_DPDT
- added JP102: FLASH/CRAM, symbol symbols:Jumper_2
- added R114, R115, R116: 10k, Resistor_SMD:R_0805_2012Metric, symbol Device:R
- added R117, R118: 100, Resistor_SMD:R_0805_2012Metric, symbol Device:R
- added U104: W25Q16DVSS, Package_SO:SOIC-8_5.23x5.23mm_P1.27mm, symbol symbols:W25Q16DVSS
- added U105: IS61WV25616FBLL-10TLI, Package_SO:TSOP-II-44_10.16x18.41mm_P0.8mm, symbol symbols:IS61WV25616FBLL-10TLI
- C105: renamed from C107; footprint (none) -> Capacitor_SMD:C_0805_2012Metric; Remarks (none) -> Class 1
- C106: renamed from C108; footprint (none) -> Capacitor_SMD:C_0805_2012Metric; Remarks (none) -> Class 1
- C107: renamed from C109; footprint (none) -> Capacitor_SMD:C_0805_2012Metric; Remarks (none) -> Class 1
- C108: renamed from C110; footprint (none) -> Capacitor_SMD:C_0805_2012Metric; Remarks (none) -> Class 1
- C112: value 4.7u -> 100n; footprint (none) -> Capacitor_SMD:C_0805_2012Metric
- R101, R102, R103, R104, R105, R106, R109, R110, R111, R112, R113: renamed from R?; footprint (none) -> Resistor_SMD:R_0805_2012Metric
- R107: value 0 -> 10k; footprint (none) -> Resistor_SMD:R_0805_2012Metric
- R108: footprint (none) -> Resistor_SMD:R_0805_2012Metric
- gave numbers to parts that had none: 11
- renumbered C103 to C101, J105 to J101, J101 to J102, J102 to J103, J103 to J104, J104 to J105, U103 to U101, U104 to U102, U105 to U103
Connections:
- net FT_VPHY is gone; now on an unnamed net: C112.1
- net GNDD is gone; now on net AGND: U101.12 (DGND), U102.12 (DGND)
- net +3V3D: no longer U101.16 (VDRIVE), U102.16 (VDRIVE)
- net AGND: now also J101.4 (GND), J101.5 (Shield), J106.2 (Ext), J107.2 (Ext), U103.103 (GND), U103.13 (GND), U103.132 (GND), U103.14 (GND), U103.140 (GND), U103.5 (GND), U103.59 (GND), U103.69 (GND), U103.86 (GND), U104.4 (GND)
- net FT_+3V3: no longer R108.1
- net FT_IO1: now also U103.61 (IOB_96)
- net FT_IO2: now also U103.62 (IOB_102)
- net FT_SPI.MISO: now also JP101.3 (C)
- net FT_SPI.MOSI: now also JP101.1 (A)
- net FT_SPI.SCK: now also U103.70 (IOB_107_SCK), U104.6 (CLK)
- net FT_SPI.~{CS}: now also U103.71 (IOB_108_SS), JP102.1 (A)
- net power_supply/IN_VBUS: now also J101.1 (VBUS)
- net FTDI/USB_DM: now reaches J101.2 (D-)
- net +3.3VD: now reaches R107.1
- net +3.3VD: now also R108.1, U101.16 (VDRIVE), U102.16 (VDRIVE), U103.100 (VCCIO_1), U103.108 (VPP_2V5), U103.46 (VCCIO_2), U103.57 (VCCIO_2), U103.72 (VCC_SPI), U103.89 (VCCIO_1), R114.1, R115.1, U104.8 (VCC); no longer J101.3 (D+)
- net at R107.2: now also JP102.2 (B), U104.1 (~{CS})
- net ICE_20MHZ: now reaches U103.49 (IOB_81_GBIN5)
- net QSPI_IO2: now reaches U103.63 (IOB_103_CBSEL0)
- net QSPI_IO2: now also R108.2, U104.3 (~{WP}/IO2)
- net QSPI_IO3: now reaches U103.64 (IOB_104_CBSEL1)
- net QSPI_IO3: now also R114.2, U104.7 (~{HOLD}/IO3)
- net FIFO.~{OE}: now reaches U103.73 (IOR_109)
- net FIFO.CLKOUT: now reaches U103.74 (IOR_110)
- net FIFO.SIWU: now reaches U103.75 (IOR_111)
- net FIFO.~{WR}: now reaches U103.76 (IOR_112)
- net FIFO.~{RD}: now reaches U103.78 (IOR_114)
- net FIFO.~{TXE}: now reaches U103.79 (IOR_115)
- net FIFO.~{RXF}: now reaches U103.80 (IOR_116)
- net FIFO.D7: now reaches U103.81 (IOR_117)
- net FIFO.D6: now reaches U103.82 (IOR_118)
- net FIFO.D5: now reaches U103.83 (IOR_119)
- net FIFO.D4: now reaches U103.84 (IOR_120)
- net FIFO.D3: now reaches U103.85 (IOR_128)
- net FIFO.D2: now reaches U103.87 (IOR_136)
- net FIFO.D1: now reaches U103.88 (IOR_137)
- net FIFO.D0: now reaches U103.90 (IOR_138)
- net +1.2VD: now reaches U103.111 (VCC), U103.27 (VCC), U103.40 (VCC), U103.92 (VCC)
- net +1.2VD: now also R117.2, R118.2
- net at U103.126 (VCCPLL1): now also C109.1, C110.1, R117.1
- net at U103.127 (GNDPLL1): now also C109.2, C110.2
- net at U103.53 (GNDPLL0): now also C112.2, C111.2
- net at U103.54 (VCCPLL0): now also C111.1, R118.1
- net ICE_CDONE: now reaches U103.65 (CDONE)
- net ICE_CDONE: now also R116.2
- net ICE_~{CRESET}: now reaches U103.66 (~{CRESET})
- net ICE_~{CRESET}: now also R115.2
- net at U103.67 (IOB_105_SDO): now also JP101.2 (B), U104.5 (DI/IO0)
- net at U103.68 (IOB_106_SDI): now also JP101.4 (D), U104.2 (DO/IO1)
- net +2V5A renamed +2.5VA
- removed net GND: C112.2, J101.4 (GND), J101.5 (Shield), J106.2 (Ext), J107.2 (Ext), U103.103 (GND), U103.13 (GND), U103.132 (GND), U103.14 (GND), U103.140 (GND), U103.5 (GND), U103.59 (GND), U103.69 (GND), U103.86 (GND)
- new net: U105.11 (VDD), U105.33 (VDD)
- new net: U105.12 (GND), U105.34 (GND)
- new net FTDI/USB_DP: J101.3 (D+)
- new net FT_3V3: R116.1
Other:
- added sheet FTDI (ftdi.kicad_sch)
- sheet Input Amplifier 1 ports: added none; removed +2V5A, +3V3A
- sheet Input Amplifier 2 ports: added none; removed +2V5A, +3V3A
- sheet Input Amplifier 3 ports: added none; removed +2V5A, +3V3A
- sheet Input Amplifier 4 ports: added none; removed +2V5A, +3V3A
- sheet power_supply ports: added PGOOD; removed none
- note removed: "USB inrush current limit: 50uC charge transferred by current _exceeding_ 100mA"
- moved on the sheet: C101, C102, C103, C104, C105, C106, C107, C108, D101, D102, D103, D104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

Commit message: Schematic sketching done
Parts:
- removed C102, C103, C104: 10u/10v, symbol Device:C_Polarized
- removed C106, C107, C108: 100n, Capacitor_SMD:C_0805_2012Metric, symbol Device:C
- removed D101: IN1:R,G, LED_THT:LED_D3.0mm-3, symbol Device:LED_Dual_KKA
- removed D102: IN3:R,G, LED_THT:LED_D3.0mm-3, symbol Device:LED_Dual_KKA
- removed D103: STATUS:R,G, LED_THT:LED_D3.0mm-3, symbol Device:LED_Dual_KKA
- removed D104: IN2:R,G, LED_THT:LED_D3.0mm-3, symbol Device:LED_Dual_KKA
- removed D105: IN4:R,G, LED_THT:LED_D3.0mm-3, symbol Device:LED_Dual_KKA
- removed D106: USB:G, symbol Device:LED
- removed R102, R103, R104, R105, R106, R109, R110, R111, R112, R113: 1k, Resistor_SMD:R_0805_2012Metric, symbol Device:R
- added C? (x3): 10u, symbol Device:C_Polarized
- added C? (x3): 100n, Capacitor_SMD:C_0805_2012Metric, symbol Device:C
- added D? (x6): WP130WCP/2EGW, symbol symbols:WP130WCP/2EGW
- added R? (x11): 240, Resistor_SMD:R_0805_2012Metric, symbol Device:R
- C101: value 10u/10v -> 10u; Spec1 (none) -> 16V; Spec2 (none) -> LL-ELCO
- C105: Remarks Class 1 -> (none); Spec1 (none) -> 10V; Spec2 (none) -> U2J; Tolerance (none) -> 10%
- R101: value 1k -> 220; Tolerance (none) -> 5%
- R108: renamed from R107; Tolerance (none) -> 5%
- R109: renamed from R108; Tolerance (none) -> 5%
- R115: renamed from R114; Tolerance (none) -> 5%
- R116: renamed from R115; Tolerance (none) -> 5%
- R117: renamed from R116; Tolerance (none) -> 5%
- R118: renamed from R117; Tolerance (none) -> 5%
- R119: renamed from R118; Tolerance (none) -> 5%
Connections:
- net FT_3V3 is gone; now on net +3.3VD: R117.1
- net ICE_20MHZ is gone; now on net ICE_CLK_20MHZ: U103.49 (IOB_81_GBIN5)
- net +3.3VD: now also U103.123 (VCCIO_0), U103.131 (VCCIO_0), U103.30 (VCCIO_3), U103.6 (VCCIO_3), U105.11 (VDD), U105.33 (VDD), R?.1
- net AGND: now also U105.12 (GND), U105.34 (GND), C?.2, C?.2, C?.2, C?.2, C?.2, C?.2, D?.2 (K1), D?.2 (K1), D?.2 (K1), D?.5 (K2), D?.5 (K2), D?.5 (K2)
- net FT_SPI.MOSI: now also R101.1; no longer JP101.1 (A)
- net at U103.67 (IOB_105_SDO), U104.5 (DI/IO0): now also JP101.1 (A); no longer JP101.2 (B)
- net at U101.6 (REFB): now also C?.1, C?.1
- net SRAM.A17: now reaches U103.1 (IOL_2A)
- net SRAM.A17: now also U105.44 (A17)
- net SRAM.D14: now reaches U103.10 (IOL_5B)
- net SRAM.D14: now also U105.37 (I/O14)
- net SRAM.D13: now reaches U103.11 (IOL_8A)
- net SRAM.D13: now also U105.36 (I/O13)
- net SRAM.D12: now reaches U103.12 (IOL_8B)
- net SRAM.D12: now also U105.35 (I/O12)
- net ADC1.SCK: now reaches U103.15 (IOL_10A)
- net ADC1.SCK: now also U101.15 (SCLK), U102.15 (SCLK), U103.20 (IOL_13B_GBIN7)
- net ADC1.DA: now reaches U103.16 (IOL_10B)
- net ADC1.DA: now also U101.14 (SDATAA)
- net ADC1.DB: now reaches U103.17 (IOL_12A)
- net ADC1.DB: now also U101.13 (SDATAB)
- net ADC1.~{CS}: now reaches U103.18 (IOL_12B)
- net ADC1.~{CS}: now also U101.10 (~{CS})
- net SRAM.A16: now reaches U103.2 (IOL_2B)
- net SRAM.A16: now also U105.43 (A16)
- net ADC2.DA: now reaches U103.21 (IOL_14A_GBIN6)
- net ADC2.DA: now also U102.14 (SDATAA)
- net ADC2.DB: now reaches U103.22 (IOL_14B)
- net ADC2.DB: now also U102.13 (SDATAB)
- net ADC2.~{CS}: now reaches U103.23 (IOL_17A)
- net ADC2.~{CS}: now also U102.10 (~{CS})
- net LED_IN1R: now reaches U103.24 (IOL_17B)
- net LED_IN1R: now also R?.1
- net LED_IN1G: now reaches U103.25 (IOL_18A)
- net LED_IN1G: now also R?.1
- net LED_IN2R: now reaches U103.26 (IOL_18B)
- net LED_IN2R: now also R?.1
- net LED_IN2G: now reaches U103.28 (IOL_23A)
- net LED_IN2G: now also R?.1
- net LED_IN3R: now reaches U103.29 (IOL_23B)
- net LED_IN3R: now also R?.1
- net SRAM.A15: now reaches U103.3 (IOL_3A)
- net SRAM.A15: now also U105.42 (A15)
- net LED_IN3G: now reaches U103.31 (IOL_24A)
- net LED_IN3G: now also R?.1
- net LED_IN4R: now reaches U103.32 (IOL_24B)
- net LED_IN4R: now also R?.1
- net LED_IN4G: now reaches U103.33 (IOL_25A)
- net LED_IN4G: now also R?.1
- net EXTIO8: now reaches U103.34 (IOL_25B)
- net SRAM.~{OE}: now reaches U103.4 (IOL_3B)
- net SRAM.~{OE}: now also U105.41 (~{OE})
- net SRAM.~{UB}: now reaches U103.7 (IOL_4A)
- net SRAM.~{UB}: now also U105.40 (~{UB})
- net SRAM.~{LB}: now reaches U103.8 (IOL_4B)
- net SRAM.~{LB}: now also U105.39 (~{LB})
- net SRAM.D15: now reaches U103.9 (IOL_5A)
- net SRAM.D15: now also U105.38 (I/O15)
- net SRAM.A0: now reaches U105.1 (A0)
- net SRAM.A0: now also U103.144 (IOT_222)
- net SRAM.D3: now reaches U105.10 (I/O3)
- net SRAM.D3: now also U103.134 (IOT_212)
- net SRAM.D4: now reaches U105.13 (I/O4)
- net SRAM.D4: now also U103.120 (IOT_179)
- net SRAM.D5: now reaches U105.14 (I/O5)
- net SRAM.D5: now also U103.119 (IOT_178)
- net SRAM.D6: now reaches U105.15 (I/O6)
- net SRAM.D6: now also U103.118 (IOT_177)
- net SRAM.D7: now reaches U105.16 (I/O7)
- net SRAM.D7: now also U103.117 (IOT_174)
- net SRAM.~{WE}: now reaches U105.17 (~{WE})
- net SRAM.~{WE}: now also U103.116 (IOT_173)
- net SRAM.A5: now reaches U105.18 (A5)
- net SRAM.A5: now also U103.115 (IOT_172)
- net SRAM.A6: now reaches U105.19 (A6)
- net SRAM.A6: now also U103.114 (IOT_171)
- net SRAM.A1: now reaches U105.2 (A1)
- net SRAM.A1: now also U103.143 (IOT_221)
- net SRAM.A7: now reaches U105.20 (A7)
- net SRAM.A7: now also U103.113 (IOT_170)
- net SRAM.A8: now reaches U105.21 (A8)
- net SRAM.A8: now also U103.112 (IOT_169)
- net SRAM.A9: now reaches U105.22 (A9)
- net SRAM.A9: now also U103.110 (IOT_168)
- net SRAM.A10: now reaches U105.23 (A10)
- net SRAM.A10: now also U103.107 (IOR_167)
- net SRAM.A11: now reaches U105.24 (A11)
- net SRAM.A11: now also U103.106 (IOR_166)
- net SRAM.A12: now reaches U105.25 (A12)
- net SRAM.A12: now also U103.105 (IOR_165)
- net SRAM.A13: now reaches U105.26 (A13)
- net SRAM.A13: now also U103.104 (IOR_164)
- net SRAM.A14: now reaches U105.27 (A14)
- net SRAM.A14: now also U103.102 (IOR_161)
- net SRAM.D8: now reaches U105.29 (I/O8)
- net SRAM.D8: now also U103.101 (IOR_160)
- net SRAM.A2: now reaches U105.3 (A2)
- net SRAM.A2: now also U103.142 (IOT_220)
- net SRAM.D9: now reaches U105.30 (I/O9)
- net SRAM.D9: now also U103.99 (IOR_152)
- net SRAM.D10: now reaches U105.31 (I/O10)
- net SRAM.D10: now also U103.98 (IOR_148)
- net SRAM.D11: now reaches U105.32 (I/O11)
- net SRAM.D11: now also U103.97 (IOR_147)
- net SRAM.A3: now reaches U105.4 (A3)
- net SRAM.A3: now also U103.141 (IOT_219)
- net SRAM.A4: now reaches U105.5 (A4)
- net SRAM.A4: now also U103.139 (IOT_217)
- net SRAM.~{CS}: now reaches U105.6 (~{CS})
- net SRAM.~{CS}: now also U103.138 (IOT_216)
- net SRAM.D0: now reaches U105.7 (I/O0)
- net SRAM.D0: now also U103.137 (IOT_215)
- net SRAM.D1: now reaches U105.8 (I/O1)
- net SRAM.D1: now also U103.136 (IOT_214)
- net SRAM.D2: now reaches U105.9 (I/O2)
- net SRAM.D2: now also U103.135 (IOT_213)
- net EXTIO7: now reaches U103.37 (IOB_56)
- net EXTIO6: now reaches U103.38 (IOB_57)
- net EXTIO5: now reaches U103.39 (IOB_61)
- net EXTIO4: now reaches U103.41 (IOB_63)
- net EXTIO3: now reaches U103.42 (IOB_64)
- net EXTIO2: now reaches U103.43 (IOB_71)
- net EXTIO1: now reaches U103.44 (IOB_72)
- net VCXO_DIN: now reaches U103.45 (IOB_73)
- net VCXO_SCK: now reaches U103.47 (IOB_79)
- net VCXO_~{SYNC}: now reaches U103.48 (IOB_80)
- net ICE_CLK_20MHZ: now reaches U103.52 (IOB_82_GBIN4)
- net ICE_CLK_OUT_SEL: now reaches U103.55 (IOB_91)
- net ICE_CLK_OUT: now reaches U103.56 (IOB_94)
- net ICE_REF_IN: now reaches U103.60 (IOB_95)
- net at U102.6 (REFB): now also C?.1, C?.1
- net at U102.3 (REFA): now also C?.1, C?.1
- net LED_STS_R: now reaches U103.93 (IOR_140_GBIN3)
- net LED_STS_R: now also R?.1
- net LED_STS_G: now reaches U103.94 (IOR_141_GBIN2)
- net LED_STS_G: now also R?.1
- net ~{LED_IN1R}: no longer names the net of R101.2
- net ~{LED_IN1R}: now also JP101.2 (B)
- new net: D?.4 (A21), R?.2 (x2)
- new net: D?.1 (A11), R?.2 (x3)
- new net: D?.3 (A12), R?.2 (x3)
- new net: D?.6 (A22), R?.2 (x3)
Other:
- added sheet Extension Connector (extconn.kicad_sch)
- sheet VCXO ports: added DIN, SCK, ~{SYNC}; removed DAC{DIN SCK ~{SYNC}}
- moved on the sheet: C109, C110, C111, C112, J101, J106, J107, JP101, JP102, R108, R109, R115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

Commit message: Update schematic layout, separate into sheets
Parts:
- removed C101, C109, C111, C? (x3): 10u, symbol Device:C_Polarized
- removed C105, C110, C112, C? (x3): 100n, Capacitor_SMD:C_0805_2012Metric, symbol Device:C
- removed JP101: FLASH/CRAM, symbol symbols:Jumper_4_DPDT
- removed JP102: FLASH/CRAM, symbol symbols:Jumper_2
- removed R101: 220, Resistor_SMD:R_0805_2012Metric, symbol Device:R
- removed R108, R109, R115, R116, R117: 10k, Resistor_SMD:R_0805_2012Metric, symbol Device:R
- removed R118, R119: 100, Resistor_SMD:R_0805_2012Metric, symbol Device:R
- removed U101, U102: AD7357xRU, Package_SO:TSSOP-16_4.4x5mm_P0.65mm, symbol symbols:AD7357xRU
- removed U103: ICE40HX4K, Package_QFP:TQFP-144_20x20mm_P0.5mm, symbol FPGA_Lattice:ICE40HX4K-TQ144
- removed U104: W25Q16DVSS, Package_SO:SOIC-8_5.23x5.23mm_P1.27mm, symbol symbols:W25Q16DVSS
- removed U105: IS61WV25616FBLL-10TLI, Package_SO:TSOP-II-44_10.16x18.41mm_P0.8mm, symbol symbols:IS61WV25616FBLL-10TLI
- gave numbers to parts that had none: 14
- renumbered J102 to J101, J103 to J102, J104 to J103, J105 to J104, J101 to J105, J107 to J106, J106 to J107
Connections:
- net AGND renamed GND
- net LED_IN1G renamed LED.IN_G1
- net LED_IN1R renamed LED.IN_R1
- net LED_IN2G renamed LED.IN_G3
- net LED_IN2R renamed LED.IN_R3
- net LED_IN3G renamed LED.IN_G2
- net LED_IN3R renamed LED.IN_R2
- net LED_IN4G renamed LED.IN_G4
- net LED_IN4R renamed LED.IN_R4
- net LED_STS_G renamed LED.STS_G
- net LED_STS_R renamed LED.STS_R
Other:
- sheet clk_out renamed Clock Output
- sheet power_supply renamed Power Supply
- sheet ref_in renamed Reference Clock Input
- added sheet ADC1 (adc.kicad_sch)
- added sheet ADC2 (adc.kicad_sch)
- added sheet FPGA (fpga.kicad_sch)
- sheet FTDI ports: added IOB{~{CRESET} CDONE IO1 IO2}; removed CDONE, IO1, IO2, ~{CRESET}
- sheet VCXO ports: added DAC{DIN SCK ~{SYNC}}; removed DIN, SCK, ~{SYNC}
- note added: "G"
- note added: "IN1"
- note added: "IN2"
- note added: "IN3"
- note added: "IN4"
- note added: "PWR"
- note added: "R"
- note added: "STATUS"
- company: (none) -> R. Dobrodii
- title: (none) -> LWDO-SDR
- moved on the sheet: D101A, D101B, D102A, D102B, D103A, D103B, J101, J102, J103, J104, J105, J106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
