File: lwdo-sdr.kicad_sch (KiCad schematic)
At the start: 21 parts, among them J101 IN1, J102 IN2, J103 IN3, J104 IN4, J105 USB_B, J106 CLK_OUT, J107 REF_IN

Commit message: Schematic: change order of level indicator LEDs from 1-3-2-4 to 1-2-3-4
Connections:
- net LED.IN_G2: now also R107.1; no longer R109.1
- net LED.IN_G3: now also R109.1; no longer R107.1
- net LED.IN_R2: now also R106.1; no longer R108.1
- net LED.IN_R3: now also R108.1; no longer R106.1
Changed lines of the file:
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@@
     (stroke (width 0) (type default) (color 0 0 0 0))
   )
-  (text "IN3" (at 375.92 175.26 0)
+  (text "IN3" (at 375.92 200.66 0)
     (effects (font (size 1.27 1.27)) (justify left bottom))
   )
@@
     (effects (font (size 1.27 1.27)) (justify left bottom))
   )
-  (text "IN2" (at 375.92 200.66 0)
+  (text "IN2" (at 375.92 175.26 0)
     (effects (font (size 1.27 1.27)) (justify left bottom))
   )
@@
     (effects (font (size 1.27 1.27)) (justify left bottom))
   )
-  (label "LED.IN_G3" (at 339.09 180.34 0)
+  (label "LED.IN_G3" (at 339.09 205.74 0)
     (effects (font (size 1.27 1.27)) (justify left bottom))
   )
-  (label "LED.IN_R3" (at 339.09 175.26 0)
+  (label "LED.IN_R3" (at 339.09 200.66 0)
     (effects (font (size 1.27 1.27)) (justify left bottom))
   )
@@
     (effects (font (size 1.27 1.27)) (justify left bottom))
   )
-  (label "LED.IN_G2" (at 339.09 205.74 0)
+  (label "LED.IN_G2" (at 339.09 180.34 0)
     (effects (font (size 1.27 1.27)) (justify left bottom))
   )
@@
     (effects (font (size 1.27 1.27)) (justify right bottom))
   )
-  (label "LED.IN_R2" (at 339.09 200.66 0)
+  (label "LED.IN_R2" (at 339.09 175.26 0)
     (effects (font (size 1.27 1.27)) (justify left bottom))
   )

Commit message: Schematic: add PNs for resistors
Parts:
- R101, R102, R103, R104, R105, R106, R107, R108, R109, R110, R111: Mfr (none) -> Bourns; Mfr PN (none) -> CR0805-FX-2200ELF
Changed lines of the file:
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@@
+      (effects (font (size 1.27 1.27)) hide)
+    )
+    (property "Mfr" "Bourns" (id 5) (at 355.6 226.06 0)
+      (effects (font (size 1.27 1.27)) hide)
+    )
+    (property "Mfr PN" "CR0805-FX-2200ELF" (id 6) (at 355.6 226.06 0)
       (effects (font (size 1.27 1.27)) hide)
     )
@@
       (effects (font (size 1.27 1.27)) hide)
     )
+    (property "Mfr" "Bourns" (id 5) (at 355.6 200.66 0)
+      (effects (font (size 1.27 1.27)) hide)
+    )
+    (property "Mfr PN" "CR0805-FX-2200ELF" (id 6) (at 355.6 200.66 0)
+      (effects (font (size 1.27 1.27)) hide)
+    )
     (pin "1")
     (pin "2")
@@
       (effects (font (size 1.27 1.27)) hide)
     )
+    (property "Mfr" "Bourns" (id 5) (at 317.5 168.91 0)
+      (effects (font (size 1.27 1.27)) hide)
+    )
+    (property "Mfr PN" "CR0805-FX-2200ELF" (id 6) (at 317.5 168.91 0)
+      (effects (font (size 1.27 1.27)) hide)
+    )
     (pin "1")
     (pin "2")
@@
       (effects (font (size 1.27 1.27)) hide)
     )
+    (property "Mfr" "Bourns" (id 5) (at 355.6 231.14 0)
+      (effects (font (size 1.27 1.27)) hide)
+    )
+    (property "Mfr PN" "CR0805-FX-2200ELF" (id 6) (at 355.6 231.14 0)
+      (effects (font (size 1.27 1.27)) hide)
+    )
     (pin "1")
     (pin "2")
@@
       (effects (font (size 1.27 1.27)) hide)
     )
+    (property "Mfr" "Bourns" (id 5) (at 355.6 180.34 0)
+      (effects (font (size 1.27 1.27)) hide)
+    )
+    (property "Mfr PN" "CR0805-FX-2200ELF" (id 6) (at 355.6 180.34 0)
+      (effects (font (size 1.27 1.27)) hide)
+    )
     (pin "1")
     (pin "2")
@@
       (effects (font (size 1.27 1.27)) hide)
     )
+    (property "Mfr" "Bourns" (id 5) (at 355.6 175.26 0)
+      (effects (font (size 1.27 1.27)) hide)
+    )
+    (property "Mfr PN" "CR0805-FX-2200ELF" (id 6) (at 355.6 175.26 0)
+      (effects (font (size 1.27 1.27)) hide)
+    )
     (pin "1")
     (pin "2")
@@
       (effects (font (size 1.27 1.27)) hide)
     )
+    (property "Mfr" "Bourns" (id 5) (at 355.6 149.86 0)
+      (effects (font (size 1.27 1.27)) hide)
+    )
+    (property "Mfr PN" "CR0805-FX-2200ELF" (id 6) (at 355.6 149.86 0)
+      (effects (font (size 1.27 1.27)) hide)
+    )
     (pin "1")
     (pin "2")
@@
       (effects (font (size 1.27 1.27)) hide)
     )
+    (property "Mfr" "Bourns" (id 5) (at 317.5 173.99 0)
+      (effects (font (size 1.27 1.27)) hide)
+    )
+    (property "Mfr PN" "CR0805-FX-2200ELF" (id 6) (at 317.5 173.99 0)
+      (effects (font (size 1.27 1.27)) hide)
+    )
     (pin "1")
     (pin "2")
@@
       (effects (font (size 1.27 1.27)) hide)
     )
+    (property "Mfr" "Bourns" (id 5) (at 355.6 154.94 0)
+      (effects (font (size 1.27 1.27)) hide)
+    )
+    (property "Mfr PN" "CR0805-FX-2200ELF" (id 6) (at 355.6 154.94 0)
+      (effects (font (size 1.27 1.27)) hide)
+    )
     (pin "1")
     (pin "2")
@@
       (effects (font (size 1.27 1.27)) hide)
     )
+    (property "Mfr" "Bourns" (id 5) (at 317.5 199.39 0)
+      (effects (font (size 1.27 1.27)) hide)
+    )
+    (property "Mfr PN" "CR0805-FX-2200ELF" (id 6) (at 317.5 199.39 0)
+      (effects (font (size 1.27 1.27)) hide)
+    )
     (pin "1")
     (pin "2")
@@
       (effects (font (size 1.27 1.27)) hide)
     )
+    (property "Mfr" "Bourns" (id 5) (at 355.6 205.74 0)
+      (effects (font (size 1.27 1.27)) hide)
+    )
+    (property "Mfr PN" "CR0805-FX-2200ELF" (id 6) (at 355.6 205.74 0)
+      (effects (font (size 1.27 1.27)) hide)
+    )

Commit message: Combined update (kicad 6.0.4..) - Update schematic to kicad 6.0.4 - Assign footprints for SMA connectors - Replace MCP1825T with MCP1824T (chip shortages..)
Parts:
- J101, J102, J103, J104, J106, J107: footprint (none) -> Connector_Coaxial:SMA_Molex_73251-2200_Horizontal
Changed lines of the file:
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@@
     (property "Reference" "J104" (id 0) (at 63.8174 121.4736 0))
     (property "Value" "IN4" (id 1) (at 63.8174 124.0105 0))
-    (property "Footprint" "" (id 2) (at 63.5 127 0)
+    (property "Footprint" "Connector_Coaxial:SMA_Molex_73251-2200_Horizontal" (id 2) (at 63.5 127 0)
       (effects (font (size 1.27 1.27)) hide)
     )
@@
     (property "Reference" "J102" (id 0) (at 63.8174 70.6736 0))
     (property "Value" "IN2" (id 1) (at 63.8174 73.2105 0))
-    (property "Footprint" "" (id 2) (at 63.5 76.2 0)
+    (property "Footprint" "Connector_Coaxial:SMA_Molex_73251-2200_Horizontal" (id 2) (at 63.5 76.2 0)
       (effects (font (size 1.27 1.27)) hide)
     )
@@
     (property "Reference" "J101" (id 0) (at 63.8174 45.2736 0))
     (property "Value" "IN1" (id 1) (at 63.8174 47.8105 0))
-    (property "Footprint" "" (id 2) (at 63.5 50.8 0)
+    (property "Footprint" "Connector_Coaxial:SMA_Molex_73251-2200_Horizontal" (id 2) (at 63.5 50.8 0)
       (effects (font (size 1.27 1.27)) hide)
     )
@@
     (pin "2")
     (pin "3")
+    (pin "4")
+    (pin "5")
+    (pin "6")
   )
   (symbol (lib_id "Device:R") (at 355.6 200.66 90) (mirror x) (unit 1)
@@
       (effects (font (size 1.27 1.27)) hide)
     )
+    (pin "1")
+    (pin "2")
+    (pin "3")
     (pin "4")
     (pin "5")
@@
       (effects (font (size 1.27 1.27)) hide)
     )
+    (pin "1")
+    (pin "2")
+    (pin "3")
     (pin "4")
     (pin "5")
@@
       (effects (font (size 1.27 1.27)) (justify left))
     )
-    (property "Footprint" "" (id 2) (at 342.9 101.6 0)
+    (property "Footprint" "Connector_Coaxial:SMA_Molex_73251-2200_Horizontal" (id 2) (at 342.9 101.6 0)
       (effects (font (size 1.27 1.27)) hide)
     )
@@
       (effects (font (size 1.27 1.27)) hide)
     )
+    (pin "1")
+    (pin "2")
+    (pin "3")
     (pin "4")
     (pin "5")
@@
     (pin "2")
     (pin "3")
+    (pin "4")
+    (pin "5")
+    (pin "6")
   )
   (symbol (lib_id "power:GND") (at 63.5 57.15 0) (unit 1)
@@
       (effects (font (size 1.27 1.27)) (justify left))
     )
-    (property "Footprint" "" (id 2) (at 342.9 62.23 0)
+    (property "Footprint" "Connector_Coaxial:SMA_Molex_73251-2200_Horizontal" (id 2) (at 342.9 62.23 0)
       (effects (font (size 1.27 1.27)) hide)
     )
@@
     (property "Reference" "J103" (id 0) (at 63.8174 96.0736 0))
     (property "Value" "IN3" (id 1) (at 63.8174 98.6105 0))
-    (property "Footprint" "" (id 2) (at 63.5 101.6 0)
+    (property "Footprint" "Connector_Coaxial:SMA_Molex_73251-2200_Horizontal" (id 2) (at 63.5 101.6 0)
       (effects (font (size 1.27 1.27)) hide)
     )
@@
     (pin "2")
     (pin "3")
+    (pin "4")
+    (pin "5")
+    (pin "6")
   )
   (symbol (lib_id "Device:R") (at 317.5 199.39 270) (unit 1)
@@
     )
     (path "/4237216f-1980-4d4e-a9e0-4008f7caeeed"
-      (reference "J101") (unit 1) (value "IN1") (footprint "")
+      (reference "J101") (unit 1) (value "IN1") (footprint "Connector_Coaxial:SMA_Molex_73251-2200_Horizontal")
     )
     (path "/215be0a7-153a-4e22-aec6-8d9afc1b371d"
-      (reference "J102") (unit 1) (value "IN2") (footprint "")
+      (reference "J102") (unit 1) (value "IN2") (footprint "Connector_Coaxial:SMA_Molex_73251-2200_Horizontal")
     )
     (path "/bbe93777-151a-4b3d-85c8-52f7d82c6ac1"
-      (reference "J103") (unit 1) (value "IN3") (footprint "")
+      (reference "J103") (unit 1) (value "IN3") (footprint "Connector_Coaxial:SMA_Molex_73251-2200_Horizontal")
     )
     (path "/10de0316-f50c-41bc-b1a7-9e2ead88633d"
-      (reference "J104") (unit 1) (value "IN4") (footprint "")
+      (reference "J104") (unit 1) (value "IN4") (footprint "Connector_Coaxial:SMA_Molex_73251-2200_Horizontal")
     )
     (path "/11335b39-a06a-4687-a18f-a62cc5f4c31e"
@@
     )
     (path "/a3049626-42e2-4901-9209-abf8037b2db1"
-      (reference "J106") (unit 1) (value "CLK_OUT") (footprint "")
+      (reference "J106") (unit 1) (value "CLK_OUT") (footprint "Connector_Coaxial:SMA_Molex_73251-2200_Horizontal")
     )
     (path "/6bf68021-b6d9-4b68-b5d0-e7bba7266a3a"
-      (reference "J107") (unit 1) (value "REF_IN") (footprint "")
+      (reference "J107") (unit 1) (value "REF_IN") (footprint "Connector_Coaxial:SMA_Molex_73251-2200_Horizontal")
     )
     (path "/6c944c46-64bf-4c4b-bb86-1cfbfa0c92c2/0805070c-2ea9-411a-9750-9cdf6d83d8cc"
@@
     )
     (path "/b1f2a3fd-0146-428d-afd2-4c52a4413b8f/864dea59-fd13-4329-a53e-5e380eaeb6e0"
-      (reference "U1204") (unit 1) (value "MCP1825T-330") (footprint "Package_TO_SOT_SMD:SOT-223-6")
+      (reference "U1204") (unit 1) (value "MCP1824T-330") (footprint "Package_TO_SOT_SMD:SOT-223-6")
     )
     (path "/b1f2a3fd-0146-428d-afd2-4c52a4413b8f/1c1d1d5a-9d74-4ac1-8d15-82b903996c68"
@@
     )
     (path "/b1f2a3fd-0146-428d-afd2-4c52a4413b8f/09a714bb-1e4f-4ca4-875a-7ff90f22b1c1"
-      (reference "U1206") (unit 1) (value "MCP1825T-330") (footprint "Package_TO_SOT_SMD:SOT-223-6")
+      (reference "U1206") (unit 1) (value "MCP1824T-330") (footprint "Package_TO_SOT_SMD:SOT-223-6")
     )
     (path "/b1f2a3fd-0146-428d-afd2-4c52a4413b8f/282509f6-9c0f-4416-8deb-f158ad7b13d8"

Commit message: Assign WP130WCP and DTO050 footprints in schematic
Parts:
- D101, D102, D103: footprint (none) -> custom-footprints:WP130WCP
Changed lines of the file:
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@@
     (property "Reference" "D101" (id 0) (at 303.5935 161.2732 0))
     (property "Value" "WP130WCP/2EGW" (id 1) (at 303.5935 163.8101 0))
-    (property "Footprint" "" (id 2) (at 303.53 171.45 0)
+    (property "Footprint" "custom-footprints:WP130WCP" (id 2) (at 303.53 171.45 0)
       (effects (font (size 1.27 1.27)) hide)
     )
@@
     (property "Reference" "D102" (id 0) (at 369.5065 167.6232 0))
     (property "Value" "WP130WCP/2EGW" (id 1) (at 369.5065 170.1601 0))
-    (property "Footprint" "" (id 2) (at 369.57 177.8 0)
+    (property "Footprint" "custom-footprints:WP130WCP" (id 2) (at 369.57 177.8 0)
       (effects (font (size 1.27 1.27)) hide)
     )
@@
     (property "Reference" "D101" (id 0) (at 303.5935 186.6732 0))
     (property "Value" "WP130WCP/2EGW" (id 1) (at 303.5935 189.2101 0))
-    (property "Footprint" "" (id 2) (at 303.53 196.85 0)
+    (property "Footprint" "custom-footprints:WP130WCP" (id 2) (at 303.53 196.85 0)
       (effects (font (size 1.27 1.27)) hide)
     )
@@
     (property "Reference" "D103" (id 0) (at 369.5065 218.4232 0))
     (property "Value" "WP130WCP/2EGW" (id 1) (at 369.5065 220.9601 0))
-    (property "Footprint" "" (id 2) (at 369.57 228.6 0)
+    (property "Footprint" "custom-footprints:WP130WCP" (id 2) (at 369.57 228.6 0)
       (effects (font (size 1.27 1.27)) hide)
     )
@@
     (property "Reference" "D102" (id 0) (at 369.5065 142.2232 0))
     (property "Value" "WP130WCP/2EGW" (id 1) (at 369.5065 144.7601 0))
-    (property "Footprint" "" (id 2) (at 369.57 152.4 0)
+    (property "Footprint" "custom-footprints:WP130WCP" (id 2) (at 369.57 152.4 0)
       (effects (font (size 1.27 1.27)) hide)
     )
@@
     (property "Reference" "D103" (id 0) (at 369.5065 193.0232 0))
     (property "Value" "WP130WCP/2EGW" (id 1) (at 369.5065 195.5601 0))
-    (property "Footprint" "" (id 2) (at 369.57 203.2 0)
+    (property "Footprint" "custom-footprints:WP130WCP" (id 2) (at 369.57 203.2 0)
       (effects (font (size 1.27 1.27)) hide)
     )
@@
     )
     (path "/4d8f897b-6041-42de-a260-e343002ccde3"
-      (reference "D101") (unit 1) (value "WP130WCP/2EGW") (footprint "")
+      (reference "D101") (unit 1) (value "WP130WCP/2EGW") (footprint "custom-footprints:WP130WCP")
     )
     (path "/6bb6f6f7-0d75-4e60-be21-af4ac468b4b3"
-      (reference "D101") (unit 2) (value "WP130WCP/2EGW") (footprint "")
+      (reference "D101") (unit 2) (value "WP130WCP/2EGW") (footprint "custom-footprints:WP130WCP")
     )
     (path "/8513d0cf-a525-494d-8f59-c2d84b6bdbf5"
-      (reference "D102") (unit 1) (value "WP130WCP/2EGW") (footprint "")
+      (reference "D102") (unit 1) (value "WP130WCP/2EGW") (footprint "custom-footprints:WP130WCP")
     )
     (path "/576f8318-b775-488e-a91c-e5ab355014d5"
-      (reference "D102") (unit 2) (value "WP130WCP/2EGW") (footprint "")
+      (reference "D102") (unit 2) (value "WP130WCP/2EGW") (footprint "custom-footprints:WP130WCP")
     )
     (path "/d79e290a-17a4-4963-9159-0a74bf5b862e"
-      (reference "D103") (unit 1) (value "WP130WCP/2EGW") (footprint "")
+      (reference "D103") (unit 1) (value "WP130WCP/2EGW") (footprint "custom-footprints:WP130WCP")
     )
     (path "/7b8b1554-10f6-4a47-809d-60070a393a20"
-      (reference "D103") (unit 2) (value "WP130WCP/2EGW") (footprint "")
+      (reference "D103") (unit 2) (value "WP130WCP/2EGW") (footprint "custom-footprints:WP130WCP")
     )
     (path "/ce49f942-6156-4865-828b-a40f6feba933/33a6eec2-47f8-4da8-ae0b-3584f8f54022"
@@
     )
     (path "/177d13d9-9b2e-4b07-87ff-23a6a61e9b1b/3053450f-d4ed-46fe-b920-70254e8e7623"
-      (reference "X902") (unit 1) (value "DOT050V-020.0M") (footprint "")
+      (reference "X902") (unit 1) (value "DOT050V-020.0M") (footprint "custom-footprints:ConnorWinfield_DOT050")
     )
     (path "/a09bc8b0-9f2c-46ec-b332-970553d5b598/bdef7b71-ec45-4ca6-b661-4ff6d725c8cc"
