File: vcxo.kicad_sch (KiCad schematic)
At the start: 27 parts, among them U901 DAC8551, U902 MCP1501-33xSN, U903 NCS325, U904 74LVC2GU04, U905 74LVC2G04, X901 TXEAADSANF-20.0, X902 DOT050V-020.0M

Commit message: Schematic: add PNs for resistors
Parts:
- R901, R904: Mfr (none) -> Bourns; Mfr PN (none) -> CR0805-FX-1002ELF
- R902: Mfr (none) -> Bourns; Mfr PN (none) -> CR0805-FX-49R9ELF
- R903: Mfr (none) -> Bourns; Mfr PN (none) -> CR0805-FX-2401ELF
- R905: Mfr (none) -> Bourns; Mfr PN (none) -> CR0805-FX-1003ELF
Changed lines of the file:
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@@
+      (effects (font (size 1.27 1.27)) hide)
+    )
+    (property "Mfr" "Bourns" (id 5) (at 100.33 127 0)
+      (effects (font (size 1.27 1.27)) hide)
+    )
+    (property "Mfr PN" "CR0805-FX-1002ELF" (id 6) (at 100.33 127 0)
       (effects (font (size 1.27 1.27)) hide)
     )
@@
     )
     (property "Tolerance" "" (id 4) (at 106.68 69.85 0)
+      (effects (font (size 1.27 1.27)) hide)
+    )
+    (property "Mfr" "Bourns" (id 5) (at 106.68 69.85 0)
+      (effects (font (size 1.27 1.27)) hide)
+    )
+    (property "Mfr PN" "CR0805-FX-49R9ELF" (id 6) (at 106.68 69.85 0)
       (effects (font (size 1.27 1.27)) hide)
     )
@@
     )
     (property "Tolerance" "" (id 4) (at 107.95 102.87 0)
+      (effects (font (size 1.27 1.27)) hide)
+    )
+    (property "Mfr" "Bourns" (id 5) (at 107.95 102.87 0)
+      (effects (font (size 1.27 1.27)) hide)
+    )
+    (property "Mfr PN" "CR0805-FX-2401ELF" (id 6) (at 107.95 102.87 0)
       (effects (font (size 1.27 1.27)) hide)
     )
@@
       (effects (font (size 1.27 1.27)) hide)
     )
+    (property "Mfr" "Bourns" (id 5) (at 209.55 133.35 0)
+      (effects (font (size 1.27 1.27)) hide)
+    )
+    (property "Mfr PN" "CR0805-FX-1003ELF" (id 6) (at 209.55 133.35 0)
+      (effects (font (size 1.27 1.27)) hide)
+    )
     (pin "1")
     (pin "2")
@@
       (effects (font (size 1.27 1.27)) hide)
     )
+    (property "Mfr" "Bourns" (id 5) (at 200.66 125.73 0)
+      (effects (font (size 1.27 1.27)) hide)
+    )
+    (property "Mfr PN" "CR0805-FX-1002ELF" (id 6) (at 200.66 125.73 0)
+      (effects (font (size 1.27 1.27)) hide)
+    )
