File: lwdo-sdr.kicad_pcb (KiCad board)
At the start: 2 copper layers, 267 parts, among them J101 USB_B, Q901 2N7002, Q903 2N7002, U1001 AT93C56, U1002 FT2232HL, U101 AD7357xRU, U102 AD7357xRU, U103 ICE40HX4K, U104 W25Q16DVSS, U105 IS61WV25616FBLL-10TLI, U201 THS4521ID, U301 THS4521ID, U401 THS4521ID, U501 THS4521ID, U601 DAC8551, U602 MCP1501-33xSN, U603 NCS325, U604 74LVC2GU04, U605 74LVC2G04, U701 74LVC1G157, U702 74LVC2G04, U801 74LVC2GU04, U802 74LVC2G04, U901 MCP1825T-330, U902 NCV8164ASN120T1G, U903 MCP1825T-330, U904 NCV8164ASN250T1G, U905 NCV8164ASN330T1G, X601 TXEAADSANF-20.0, Y1001 12MHz

Commit message: Schematic sketching done
Parts:
- added R101: 220, Resistor_SMD:R_0805_2012Metric, F.Cu at (166.5, 138.3)
- moved U102 121.3 mm to (19.1, 118.1)
- moved U101 83.7 mm to (19.1, 110.5)
- moved C106 56.3 mm to (187.0, 81.3)
- moved C108 56.3 mm to (187.0, 78.3)
- moved C110 56.3 mm to (191.5, 78.3)
- moved C112 56.3 mm to (199.8, 72.7)
- moved C201 56.3 mm to (230.5, 96.5)
- moved C203 56.3 mm to (230.5, 93.5)
- moved C204 56.3 mm to (226.1, 96.5)
- moved C206 56.3 mm to (222.1, 103.0)
- moved C211 56.3 mm to (222.1, 100.0)
- moved C212 56.3 mm to (222.1, 106.0)
- moved C213 56.3 mm to (226.5, 99.5)
- moved C214 56.3 mm to (226.1, 93.5)
- moved C301 56.3 mm to (266.3, 70.2)
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- renumbered R101 to R102, R102 to R103, R103 to R104, R104 to R105, R105 to R106, R106 to R107, R107 to R108, R108 to R109, R109 to R110, R110 to R111, R111 to R112, R112 to R113, R113 to R114, R114 to R115, R115 to R116, R116 to R117, R117 to R118, R118 to R119
Connections:
- net /VCXO/DAC.DIN renamed /VCXO_DAC.DIN
- net /VCXO/DAC.SCK renamed /VCXO_DAC.SCK
- net /VCXO/DAC.~{SYNC} renamed /VCXO_DAC.~{SYNC}
- net /clk_out/CLK0 renamed /ICE_CLK_OUT1
- net /clk_out/CLK_SEL renamed /ICE_CLK_OUT_SEL
- net /ref_in/OUT renamed /ICE_REF_IN
- U101 pad 10: unconnected-(U101-Pad10) -> /ADC1.~{CS}
- U101 pad 13: unconnected-(U101-Pad13) -> /ADC1.DB
- U101 pad 14: unconnected-(U101-Pad14) -> /ADC1.DA
- U101 pad 15: unconnected-(U101-Pad15) -> /ADC2.SCK
- U102 pad 10: unconnected-(U102-Pad10) -> /ADC2.~{CS}
- U102 pad 13: unconnected-(U102-Pad13) -> /ADC2.DB
- U102 pad 14: unconnected-(U102-Pad14) -> /ADC2.DA
- U102 pad 15: unconnected-(U102-Pad15) -> /ADC2.SCK
- U103 pad 1: unconnected-(U103-Pad1) -> /SRAM.A17
- U103 pad 10: unconnected-(U103-Pad10) -> /SRAM.D14
- U103 pad 101: unconnected-(U103-Pad101) -> /SRAM.D8
- U103 pad 102: unconnected-(U103-Pad102) -> /SRAM.A14
- U103 pad 104: unconnected-(U103-Pad104) -> /SRAM.A13
- U103 pad 105: unconnected-(U103-Pad105) -> /SRAM.A12
- U103 pad 106: unconnected-(U103-Pad106) -> /SRAM.A11
- U103 pad 107: unconnected-(U103-Pad107) -> /SRAM.A10
- U103 pad 11: unconnected-(U103-Pad11) -> /SRAM.D13
- U103 pad 110: unconnected-(U103-Pad110) -> /SRAM.A9
- U103 pad 112: unconnected-(U103-Pad112) -> /SRAM.A8
- U103 pad 113: unconnected-(U103-Pad113) -> /SRAM.A7
- U103 pad 114: unconnected-(U103-Pad114) -> /SRAM.A6
- U103 pad 115: unconnected-(U103-Pad115) -> /SRAM.A5
- U103 pad 116: unconnected-(U103-Pad116) -> /SRAM.~{WE}
- U103 pad 117: unconnected-(U103-Pad117) -> /SRAM.D7
- U103 pad 118: unconnected-(U103-Pad118) -> /SRAM.D6
- U103 pad 119: unconnected-(U103-Pad119) -> /SRAM.D5
- U103 pad 12: unconnected-(U103-Pad12) -> /SRAM.D12
- U103 pad 120: unconnected-(U103-Pad120) -> /SRAM.D4
- U103 pad 123: Net-(U103-Pad123) -> +3.3VD
- U103 pad 131: Net-(U103-Pad123) -> +3.3VD
- U103 pad 134: unconnected-(U103-Pad134) -> /SRAM.D3
- U103 pad 135: unconnected-(U103-Pad135) -> /SRAM.D2
- U103 pad 136: unconnected-(U103-Pad136) -> /SRAM.D1
- U103 pad 137: unconnected-(U103-Pad137) -> /SRAM.D0
- U103 pad 138: unconnected-(U103-Pad138) -> /SRAM.~{CS}
- U103 pad 139: unconnected-(U103-Pad139) -> /SRAM.A4
- U103 pad 141: unconnected-(U103-Pad141) -> /SRAM.A3
- U103 pad 142: unconnected-(U103-Pad142) -> /SRAM.A2
- U103 pad 143: unconnected-(U103-Pad143) -> /SRAM.A1
- U103 pad 144: unconnected-(U103-Pad144) -> /SRAM.A0
- U103 pad 15: unconnected-(U103-Pad15) -> /ADC2.SCK
- U103 pad 16: unconnected-(U103-Pad16) -> /ADC1.DA
- U103 pad 17: unconnected-(U103-Pad17) -> /ADC1.DB
- U103 pad 18: unconnected-(U103-Pad18) -> /ADC1.~{CS}
- U103 pad 2: unconnected-(U103-Pad2) -> /SRAM.A16
- U103 pad 20: unconnected-(U103-Pad20) -> /ADC2.SCK
- U103 pad 21: unconnected-(U103-Pad21) -> /ADC2.DA
- U103 pad 22: unconnected-(U103-Pad22) -> /ADC2.DB
- U103 pad 23: unconnected-(U103-Pad23) -> /ADC2.~{CS}
- U103 pad 3: unconnected-(U103-Pad3) -> /SRAM.A15
- U103 pad 30: Net-(U103-Pad30) -> +3.3VD
- U103 pad 4: unconnected-(U103-Pad4) -> /SRAM.~{OE}
- U103 pad 49: unconnected-(U103-Pad49) -> /ICE_CLK_20MHZ
- U103 pad 6: Net-(U103-Pad30) -> +3.3VD
- U103 pad 7: unconnected-(U103-Pad7) -> /SRAM.~{UB}
- U103 pad 8: unconnected-(U103-Pad8) -> /SRAM.~{LB}
- U103 pad 9: unconnected-(U103-Pad9) -> /SRAM.D15
- U103 pad 97: unconnected-(U103-Pad97) -> /SRAM.D11
- U103 pad 98: unconnected-(U103-Pad98) -> /SRAM.D10
- U103 pad 99: unconnected-(U103-Pad99) -> /SRAM.D9
- U105 pad 1: unconnected-(U105-Pad1) -> /SRAM.A0
- U105 pad 10: unconnected-(U105-Pad10) -> /SRAM.D3
- U105 pad 11: Net-(U105-Pad11) -> +3.3VD
- U105 pad 12: Net-(U105-Pad12) -> AGND
- U105 pad 13: unconnected-(U105-Pad13) -> /SRAM.D4
- U105 pad 14: unconnected-(U105-Pad14) -> /SRAM.D5
- U105 pad 15: unconnected-(U105-Pad15) -> /SRAM.D6
- U105 pad 16: unconnected-(U105-Pad16) -> /SRAM.D7
- U105 pad 17: unconnected-(U105-Pad17) -> /SRAM.~{WE}
- U105 pad 18: unconnected-(U105-Pad18) -> /SRAM.A5
- U105 pad 19: unconnected-(U105-Pad19) -> /SRAM.A6
- U105 pad 2: unconnected-(U105-Pad2) -> /SRAM.A1
- U105 pad 20: unconnected-(U105-Pad20) -> /SRAM.A7
- U105 pad 21: unconnected-(U105-Pad21) -> /SRAM.A8
- U105 pad 22: unconnected-(U105-Pad22) -> /SRAM.A9
- U105 pad 23: unconnected-(U105-Pad23) -> /SRAM.A10
- U105 pad 24: unconnected-(U105-Pad24) -> /SRAM.A11
- U105 pad 25: unconnected-(U105-Pad25) -> /SRAM.A12
- U105 pad 26: unconnected-(U105-Pad26) -> /SRAM.A13
- U105 pad 27: unconnected-(U105-Pad27) -> /SRAM.A14
- U105 pad 29: unconnected-(U105-Pad29) -> /SRAM.D8
- U105 pad 3: unconnected-(U105-Pad3) -> /SRAM.A2
- U105 pad 30: unconnected-(U105-Pad30) -> /SRAM.D9
- U105 pad 31: unconnected-(U105-Pad31) -> /SRAM.D10
- U105 pad 32: unconnected-(U105-Pad32) -> /SRAM.D11
- U105 pad 33: Net-(U105-Pad11) -> +3.3VD
- U105 pad 34: Net-(U105-Pad12) -> AGND
- U105 pad 35: unconnected-(U105-Pad35) -> /SRAM.D12
- U105 pad 36: unconnected-(U105-Pad36) -> /SRAM.D13
- U105 pad 37: unconnected-(U105-Pad37) -> /SRAM.D14
- U105 pad 38: unconnected-(U105-Pad38) -> /SRAM.D15
- U105 pad 39: unconnected-(U105-Pad39) -> /SRAM.~{LB}
- U105 pad 4: unconnected-(U105-Pad4) -> /SRAM.A3
- U105 pad 40: unconnected-(U105-Pad40) -> /SRAM.~{UB}
- U105 pad 41: unconnected-(U105-Pad41) -> /SRAM.~{OE}
- U105 pad 42: unconnected-(U105-Pad42) -> /SRAM.A15
- U105 pad 43: unconnected-(U105-Pad43) -> /SRAM.A16
- U105 pad 44: unconnected-(U105-Pad44) -> /SRAM.A17
- U105 pad 5: unconnected-(U105-Pad5) -> /SRAM.A4
- U105 pad 6: unconnected-(U105-Pad6) -> /SRAM.~{CS}
- U105 pad 7: unconnected-(U105-Pad7) -> /SRAM.D0
- U105 pad 8: unconnected-(U105-Pad8) -> /SRAM.D1
- U105 pad 9: unconnected-(U105-Pad9) -> /SRAM.D2
- U605 pad 6: /VCXO/20MHZ_OUT1 -> /ICE_CLK_20MHZ
- U701 pad 1: /clk_out/CLK1 -> /VCXO/20MHZ_OUT2
Routing:
- net /SRAM.D12: track 0.00 -> 32.5 mm, vias 0 -> 2
- net /SRAM.D11: track 0.00 -> 32.2 mm, vias 0 -> 2
- net /SRAM.A14: track 0.00 -> 24.8 mm, vias 0 -> 2
- net /SRAM.A13: track 0.00 -> 23.6 mm, vias 0 -> 2
- net /SRAM.A12: track 0.00 -> 22.6 mm, vias 0 -> 2
- net /SRAM.A11: track 0.00 -> 21.5 mm, vias 0 -> 2
- net /SRAM.A10: track 0.00 -> 20.3 mm, vias 0 -> 2
- net +3.3VD: track 0.00 -> 10.2 mm
- net /SRAM.~{WE}: track 0.00 -> 5.51 mm
- net /SRAM.A8: track 0.00 -> 5.41 mm
- net /SRAM.A5: track 0.00 -> 5.39 mm
- net /SRAM.A9: track 0.00 -> 5.33 mm
- net /SRAM.A7: track 0.00 -> 5.29 mm
- net /SRAM.A6: track 0.00 -> 5.26 mm

Commit message: PCB: begin layout - Board edge - Al extrusion clearances - Mounting holes - Connectors - FPGA-SRAM A/D buses
Parts:
- removed C1004, C1006, C1007: 4.7u, Capacitor_SMD:C_0805_2012Metric
- removed C1005, C1008, C1009, C1010, C1011, C1012, C1013, C1014, C105, C106, C107, C108, C110, C112, C612, C614: 100n, Capacitor_SMD:C_0805_2012Metric
- removed C312, C313, C314, C412, C413, C414, C512, C513, C514: 1.5n, Capacitor_SMD:C_0805_2012Metric
- removed C613: 10n, Capacitor_SMD:C_0805_2012Metric
- removed C913: 1u, Capacitor_SMD:C_0805_2012Metric
- removed D104: IN2:R,G, LED_THT:LED_D3.0mm-3
- removed D105: IN4:R,G, LED_THT:LED_D3.0mm-3
- removed D701, D702, D802, D803, D905: BAT54J, Diode_SMD:D_SOD-323F
- removed Q901, Q903: 2N7002, Package_TO_SOT_SMD:SOT-23
- removed R1003, R1004: 0, Resistor_SMD:R_0805_2012Metric
- removed R1005, R1006, R1008, R1010, R1011, R115, R116, R117, R803, R906: 10k, Resistor_SMD:R_0805_2012Metric
- removed R1007: 2.2k, Resistor_SMD:R_0805_2012Metric
- removed R1009: 12k, Resistor_SMD:R_0805_2012Metric
- removed R112, R113, R114, R802: 1k, Resistor_SMD:R_0805_2012Metric
- removed R118, R119, R214, R215, R315, R415, R515: 100, Resistor_SMD:R_0805_2012Metric
- removed R209: 200, Resistor_SMD:R_0805_2012Metric
- removed R210, R211: 24, Resistor_SMD:R_0805_2012Metric
- removed R212, R213: 220, Resistor_SMD:R_0805_2012Metric
- removed R701: 75, Resistor_SMD:R_0805_2012Metric
- removed R702: 120, Resistor_SMD:R_0805_2012Metric
- removed R801: 49.9, Resistor_SMD:R_0805_2012Metric
- removed R804: 100k, Resistor_SMD:R_0805_2012Metric
- removed TP201, TP202, TP903, TP904, TP905, TP906, TP907, TP908: TestPoint, TestPoint:TestPoint_THTPad_D1.0mm_Drill0.5mm
- removed U101, U102: AD7357xRU, Package_SO:TSSOP-16_4.4x5mm_P0.65mm
- removed U103: ICE40HX4K, Package_QFP:TQFP-144_20x20mm_P0.5mm
- removed U104: W25Q16DVSS, Package_SO:SOIC-8_5.23x5.23mm_P1.27mm
- removed U105: IS61WV25616FBLL-10TLI, Package_SO:TSOP-II-44_10.16x18.41mm_P0.8mm
- removed U602: MCP1501-33xSN, Package_SO:SOIC-8_3.9x4.9mm_P1.27mm
- removed U603: NCS325, Package_TO_SOT_SMD:SOT-23-5
- removed U604: 74LVC2GU04, Package_TO_SOT_SMD:SOT-23-6
- removed U605, U702, U802: 74LVC2G04, Package_TO_SOT_SMD:SOT-23-6
- removed X601: TXEAADSANF-20.0, Crystal:Crystal_SMD_3225-4Pin_3.2x2.5mm
- removed Y1001: 12MHz, Crystal:Crystal_SMD_3225-4Pin_3.2x2.5mm
- added C1101: 1n, Capacitor_SMD:C_0805_2012Metric, F.Cu at (95.5, -33.2)
- added C1102: 10n, Capacitor_SMD:C_0805_2012Metric, F.Cu at (85.5, -24.5)
- added C1103: 10n, Capacitor_SMD:C_0805_2012Metric, F.Cu at (90.6, -30.2)
- added C1104: 100n, Capacitor_SMD:C_0805_2012Metric, F.Cu at (95.5, -36.2)
- added C1105: 1u, Capacitor_SMD:C_0805_2012Metric, F.Cu at (100.3, -39.1)
- added C1201: 100n, Capacitor_SMD:C_0805_2012Metric, F.Cu at (-63.0, 35.2)
- added C1202: 100n, Capacitor_SMD:C_0805_2012Metric, F.Cu at (-37.1, 8.36)
- added C1203: 100n, Capacitor_SMD:C_0805_2012Metric, F.Cu at (-63.0, 32.2)
- added C1204: 100n, Capacitor_SMD:C_0805_2012Metric, F.Cu at (-57.7, 26.1)
- added C1205: 4.7u, Capacitor_SMD:C_0805_2012Metric, F.Cu at (-47.8, 16.5)
- added C1206: 4.7u, Capacitor_SMD:C_0805_2012Metric, F.Cu at (-46.5, 9.80)
- added C1207: 1u, Capacitor_SMD:C_0805_2012Metric, F.Cu at (-42.1, 9.80)
- added C1208: 100n, Capacitor_SMD:C_0805_2012Metric, F.Cu at (-46.5, 12.8)
- added C1209: 1u, Capacitor_SMD:C_0805_2012Metric, F.Cu at (-62.2, 29.1)
- added C1210: 100n, Capacitor_SMD:C_0805_2012Metric, F.Cu at (-42.1, 12.8)
- added C1211: 22u, Capacitor_SMD:CP_Elec_4x5.8, F.Cu at (-71.4, 23.3)
- added C1212: 1u, Capacitor_SMD:C_0805_2012Metric, F.Cu at (-50.2, 21.1)
- added C1213: 1u, Capacitor_SMD:C_0805_2012Metric, F.Cu at (-62.2, 26.1)
- added C1214: 1u, Capacitor_SMD:C_0805_2012Metric, F.Cu at (-37.1, 5.35)
- added C1215: 1u, Capacitor_SMD:C_0805_2012Metric, F.Cu at (-54.7, 21.1)
- added C1216: 1u, Capacitor_SMD:C_0805_2012Metric, F.Cu at (-57.7, 29.1)
- added C1217: 1u, Capacitor_SMD:C_0805_2012Metric, F.Cu at (-73.1, 35.5)
- added C1301: 27p, Capacitor_SMD:C_0805_2012Metric, F.Cu at (199.6, 113.0)
- added C1302: 27p, Capacitor_SMD:C_0805_2012Metric, F.Cu at (180.7, 127.4)
- added C1303: 4.7u, Capacitor_SMD:C_0805_2012Metric, F.Cu at (195.1, 114.2)
- added C1304: 4.7u, Capacitor_SMD:C_0805_2012Metric, F.Cu at (185.6, 123.0)
- added C1305: 100n, Capacitor_SMD:C_0805_2012Metric, F.Cu at (190.0, 121.4)
- added C1306: 100n, Capacitor_SMD:C_0805_2012Metric, F.Cu at (185.6, 126.0)
- added C1307: 100n, Capacitor_SMD:C_0805_2012Metric, F.Cu at (200.4, 104.0)
- added C1308: 4.7u, Capacitor_SMD:C_0805_2012Metric, F.Cu at (195.1, 111.2)
- added C1309: 4.7u, Capacitor_SMD:C_0805_2012Metric, F.Cu at (200.4, 107.0)
- added C1310: 100n, Capacitor_SMD:C_0805_2012Metric, F.Cu at (180.7, 130.4)
- added C1311: 100n, Capacitor_SMD:C_0805_2012Metric, F.Cu at (204.8, 107.0)
- added C1312: 100n, Capacitor_SMD:C_0805_2012Metric, F.Cu at (194.3, 118.4)
- added C1313: 100n, Capacitor_SMD:C_0805_2012Metric, F.Cu at (204.8, 104.0)
- added C1314: 100n, Capacitor_SMD:C_0805_2012Metric, F.Cu at (200.0, 110.0)
- added C1401: 100n, Capacitor_SMD:C_0805_2012Metric, F.Cu at (20.1, -64.9)
- added C1402: 100n, Capacitor_SMD:C_0805_2012Metric, F.Cu at (32.3, -66.7)
- added C1403: 100n, Capacitor_SMD:C_0805_2012Metric, F.Cu at (15.7, -64.9)
- added C1404: 4.7u, Capacitor_SMD:C_0805_2012Metric, F.Cu at (32.3, -69.7)
- added C1405: 100n, Capacitor_SMD:C_0805_2012Metric, F.Cu at (15.7, -61.9)
- added C1406: 100n, Capacitor_SMD:C_0805_2012Metric, F.Cu at (24.6, -64.9)
- added C202: 4.7u, Capacitor_SMD:C_0805_2012Metric, F.Cu at (-62.7, -1.56)
- added C215: 100n, Capacitor_SMD:C_0805_2012Metric, F.Cu at (-47.8, -5.94)
- added C216: 100n, Capacitor_SMD:C_0805_2012Metric, F.Cu at (-34.5, -21.6)
- added C217: 100n, Capacitor_SMD:C_0805_2012Metric, F.Cu at (-34.5, -24.6)
- added C218: 100n, Capacitor_SMD:C_0805_2012Metric, F.Cu at (-30.0, -15.5)
- added C219: 100n, Capacitor_SMD:C_0805_2012Metric, F.Cu at (-38.9, -5.77)
- added C220: 10u, Capacitor_SMD:CP_Elec_4x5.8, F.Cu at (-61.1, -5.99)
- added C221: 100n, Capacitor_SMD:C_0805_2012Metric, F.Cu at (-34.5, -18.5)
- added C222: 10u, Capacitor_SMD:CP_Elec_4x5.8, F.Cu at (-47.1, -10.4)
- added C223: 100n, Capacitor_SMD:C_0805_2012Metric, F.Cu at (-36.5, -8.78)
- added C302: 6.8n, Capacitor_SMD:C_0805_2012Metric, F.Cu at (98.9, 49.0)
- added C402: 6.8n, Capacitor_SMD:C_0805_2012Metric, F.Cu at (23.0, 11.1)
- added C502: 6.8n, Capacitor_SMD:C_0805_2012Metric, F.Cu at (60.3, 4.33)
- added C602: 6.8n, Capacitor_SMD:C_0805_2012Metric, F.Cu at (114.7, -69.9)
- added C603: 6.8n, Capacitor_SMD:C_0805_2012Metric, F.Cu at (121.5, -76.3)
- added C704: 100n, Capacitor_SMD:C_0805_2012Metric, F.Cu at (83.7, -69.7)
- added C705: 4.7u, Capacitor_SMD:C_0805_2012Metric, F.Cu at (88.2, -70.4)
- added C706: 100n, Capacitor_SMD:C_0805_2012Metric, F.Cu at (92.5, -76.3)
- added C707: 100n, Capacitor_SMD:C_0805_2012Metric, F.Cu at (80.4, -63.8)
- added C708: 4.7u, Capacitor_SMD:C_0805_2012Metric, F.Cu at (76.0, -60.8)
- added C806: 100n, Capacitor_SMD:C_0805_2012Metric, F.Cu at (52.8, -60.8)
- added C807: 100n, Capacitor_SMD:C_0805_2012Metric, F.Cu at (65.0, -70.4)
- added C808: 4.7u, Capacitor_SMD:C_0805_2012Metric, F.Cu at (57.3, -63.8)
- added C907: 4.7u, Capacitor_SMD:C_0805_2012Metric, F.Cu at (-5.40, -11.0)
- added D1001: BAT54J, Diode_SMD:D_SOD-323F, F.Cu at (35.7, -32.4)
- added D1002: BAT54J, Diode_SMD:D_SOD-323F, F.Cu at (25.9, -20.7)
- added D1003: PESD5V0X1BT, Package_TO_SOT_SMD:SOT-23, F.Cu at (31.0, -24.4)
- added D1101: PESD5V0X1BT, Package_TO_SOT_SMD:SOT-23, F.Cu at (90.8, -34.0)
- added D1102: BAT54J, Diode_SMD:D_SOD-323F, F.Cu at (95.6, -39.2)
- added D1103: BAT54J, Diode_SMD:D_SOD-323F, F.Cu at (85.8, -27.5)
- added D1201: PTVS5V0S1UR, Diode_SMD:Nexperia_CFP3_SOD-123W, F.Cu at (-52.0, 8.87)
- added D1202: PTVS5V0S1UR, Diode_SMD:Nexperia_CFP3_SOD-123W, F.Cu at (-57.8, 5.52)
- added D1203: SBR3U40S1F, Diode_SMD:D_SOD-123F, F.Cu at (-72.4, 27.9)
- added D1204: SBR3U40S1F, Diode_SMD:D_SOD-123F, F.Cu at (-62.4, 15.2)
- added D1205: PTVS3V3S1UR, Diode_SMD:Nexperia_CFP3_SOD-123W, F.Cu at (-52.0, 5.52)
- added D1206: SBR3U40S1F, Diode_SMD:D_SOD-123F, F.Cu at (-64.7, 22.0)
- added D1207: SBR3U40S1F, Diode_SMD:D_SOD-123F, F.Cu at (-57.8, 8.87)
- added D1301: PESD2USB3UV, Package_TO_SOT_SMD:SOT-23, F.Cu at (180.9, 123.7)
- added D1401: PTVS3V3S1UR, Diode_SMD:Nexperia_CFP3_SOD-123W, F.Cu at (4.33, -41.0)
- added D301: SD12C, Diode_SMD:D_SOD-323, F.Cu at (94.9, 44.6)
- added D302: BAT54J, Diode_SMD:D_SOD-323F, F.Cu at (109.2, 42.4)
- added D303: BAT54J, Diode_SMD:D_SOD-323F, F.Cu at (111.5, 42.4)
- added D401: SD12C, Diode_SMD:D_SOD-323, F.Cu at (25.1, 4.76)
- added D402: BAT54J, Diode_SMD:D_SOD-323F, F.Cu at (18.3, 11.2)
- added D403: BAT54J, Diode_SMD:D_SOD-323F, F.Cu at (19.4, 8.11)
- added D501: SD12C, Diode_SMD:D_SOD-323, F.Cu at (62.3, -2.06)
- added D502: BAT54J, Diode_SMD:D_SOD-323F, F.Cu at (55.5, 4.39)
- added D503: BAT54J, Diode_SMD:D_SOD-323F, F.Cu at (56.7, 1.29)
- added D601: SD12C, Diode_SMD:D_SOD-323, F.Cu at (116.7, -76.3)
- added D602: BAT54J, Diode_SMD:D_SOD-323F, F.Cu at (109.9, -69.8)
- added D603: BAT54J, Diode_SMD:D_SOD-323F, F.Cu at (111.1, -72.9)
- added F1201: 1206L050/15, Fuse:Fuse_1206_3216Metric, F.Cu at (-56.7, 12.2)
- added F1202: 1206L050/15, Fuse:Fuse_1206_3216Metric, F.Cu at (-62.5, 18.5)
- added FB1001: 782853701, Inductor_SMD:L_0805_2012Metric, F.Cu at (30.5, -28.0)
- added FB1201: 782853701, Inductor_SMD:L_0805_2012Metric, F.Cu at (-57.1, 18.0)
- added FB1202: 782853701, Inductor_SMD:L_0805_2012Metric, F.Cu at (-57.1, 15.2)
- added FB1301: 782853701, Inductor_SMD:L_0805_2012Metric, F.Cu at (189.6, 118.3)
- added FB1302: 782853701, Inductor_SMD:L_0805_2012Metric, F.Cu at (195.3, 108.3)
- added FB1401: 782853701, Inductor_SMD:L_0805_2012Metric, F.Cu at (33.4, -76.4)
- added FB901: 782853701, Inductor_SMD:L_0805_2012Metric, F.Cu at (8.31, -31.9)
- added H101: MountingHole_Pad, MountingHole:MountingHole_3.2mm_M3_Pad, F.Cu at (235.0, 37.0)
- added H102: MountingHole_Pad, MountingHole:MountingHole_3.2mm_M3_Pad, F.Cu at (235.0, 143.0)
- added H103: MountingHole_Pad, MountingHole:MountingHole_3.2mm_M3_Pad, F.Cu at (87.0, 143.0)
- added H104: MountingHole_Pad, MountingHole:MountingHole_3.2mm_M3_Pad, F.Cu at (87.0, 37.0)
- added H105: MountingHole_Pad, MountingHole:MountingHole_3.2mm_M3_Pad, F.Cu at (161.0, 90.0)
- added J102: IN2, custom-footprints:SMA_Superbat_S01-ROPT4-11BS00, F.Cu at (87.6, 69.8)
- added J103: IN3, custom-footprints:SMA_Superbat_S01-ROPT4-11BS00, F.Cu at (87.6, 92.7)
- added J104: IN4, custom-footprints:SMA_Superbat_S01-ROPT4-11BS00, F.Cu at (87.6, 115.6)
- added J105: USB_B, Connector_USB:USB_B_Lumberg_2411_02_Horizontal, F.Cu at (228.7, 71.4)
- added J106: CLK_OUT, custom-footprints:SMA_Superbat_S01-ROPT4-11BS00, F.Cu at (234.4, 127.0)
- added J107: REF_IN, custom-footprints:SMA_Superbat_S01-ROPT4-11BS00, F.Cu at (234.4, 101.6)
- added J1401: Conn_02x10_Odd_Even, Connector_IDC:IDC-Header_2x10_P2.54mm_Vertical, F.Cu at (6.70, -71.6)
- added JP1001: DC, Connector_PinHeader_2.54mm:PinHeader_1x02_P2.54mm_Vertical, F.Cu at (25.7, -31.5)
- added JP1101: DC, Connector_PinHeader_2.54mm:PinHeader_1x02_P2.54mm_Vertical, F.Cu at (85.6, -38.3)
- added JP1201: USB_PON, Connector_PinHeader_2.54mm:PinHeader_1x03_P2.54mm_Vertical, F.Cu at (-63.0, 6.17)
- added JP201: FLASH/CRAM, Connector_PinHeader_2.54mm:PinHeader_2x02_P2.54mm_Vertical, F.Cu at (-54.9, -5.12)
- added JP202: FLASH/CRAM, Connector_PinHeader_2.54mm:PinHeader_1x02_P2.54mm_Vertical, F.Cu at (-34.4, -30.9)
- added L301: 18u, Inductor_SMD:L_1812_4532Metric_Pad1.30x3.40mm_HandSolder, F.Cu at (100.3, 44.6)
- added L401: 18u, Inductor_SMD:L_1812_4532Metric_Pad1.30x3.40mm_HandSolder, F.Cu at (12.1, 12.2)
- added L501: 18u, Inductor_SMD:L_1812_4532Metric_Pad1.30x3.40mm_HandSolder, F.Cu at (49.4, 5.39)
- added L601: 18u, Inductor_SMD:L_1812_4532Metric_Pad1.30x3.40mm_HandSolder, F.Cu at (103.8, -68.8)
- added Q1201: NX7002AK, Package_TO_SOT_SMD:SOT-23, F.Cu at (-46.7, 6.07)
- added Q1202: PMN48XP, Package_TO_SOT_SMD:SOT-23-6, F.Cu at (-52.4, 17.3)
- added R1101: 49.9, Resistor_SMD:R_0805_2012Metric, F.Cu at (85.5, -21.6)
- added R1102: 1k, Resistor_SMD:R_0805_2012Metric, F.Cu at (99.9, -36.2)
- added R1103: 10k, Resistor_SMD:R_0805_2012Metric, F.Cu at (95.1, -30.2)
- added R1104: 100k, Resistor_SMD:R_0805_2012Metric, F.Cu at (90.5, -27.3)
- added R1201: 1k, Resistor_SMD:R_0805_2012Metric, F.Cu at (-48.9, 24.1)
- added R1202: 2.4k, Resistor_SMD:R_0805_2012Metric, F.Cu at (-58.6, 32.1)
- added R1203: 1k, Resistor_SMD:R_0805_2012Metric, F.Cu at (-53.3, 24.1)
- added R1204: 2.4k, Resistor_SMD:R_0805_2012Metric, F.Cu at (-48.9, 27.0)
- added R1205: 220, Resistor_SMD:R_0805_2012Metric, F.Cu at (-41.4, 18.7)
- added R1206: 2.4k, Resistor_SMD:R_0805_2012Metric, F.Cu at (-45.8, 19.5)
- added R1207: 100k, Resistor_SMD:R_0805_2012Metric, F.Cu at (-53.3, 30.0)
- added R1208: 10k, Resistor_SMD:R_0805_2012Metric, F.Cu at (-58.6, 35.1)
- added R1209: 10k, Resistor_SMD:R_0805_2012Metric, F.Cu at (-53.3, 27.0)
- added R1210: 10k, Resistor_SMD:R_0805_2012Metric, F.Cu at (-39.0, 15.8)
- added R1211: 10k, Resistor_SMD:R_0805_2012Metric, F.Cu at (-43.4, 15.8)
- added R1212: 10k, Resistor_SMD:R_0805_2012Metric, F.Cu at (-37.7, 11.3)
- added R1301: 5.1k, Resistor_SMD:R_0805_2012Metric, F.Cu at (204.4, 110.0)
- added R1302: 10k, Resistor_SMD:R_0805_2012Metric, F.Cu at (185.1, 131.9)
- added R1303: 0, Resistor_SMD:R_0805_2012Metric, F.Cu at (209.2, 106.9)
- added R1304: 0, Resistor_SMD:R_0805_2012Metric, F.Cu at (225.2, 86.2)
- added R1305: 10k, Resistor_SMD:R_0805_2012Metric, F.Cu at (199.5, 116.0)
- added R1306: 2.4k, Resistor_SMD:R_0805_2012Metric, F.Cu at (204.0, 113.0)
- added R1307: 10k, Resistor_SMD:R_0805_2012Metric, F.Cu at (194.4, 121.4)
- added R1308: 12k, Resistor_SMD:R_0805_2012Metric, F.Cu at (185.1, 129.0)
- added R1309: 10k, Resistor_SMD:R_0805_2012Metric, F.Cu at (190.0, 124.4)
- added R1310: 10k, Resistor_SMD:R_0805_2012Metric, F.Cu at (208.8, 110.0)
- added R1311: 10k, Resistor_SMD:R_0805_2012Metric, F.Cu at (209.2, 104.0)
- added R1401: 0, Resistor_SMD:R_0805_2012Metric, F.Cu at (20.1, -61.9)
- added R1402: DNP, Resistor_SMD:R_0805_2012Metric, F.Cu at (15.6, -50.1)
- added R1403: 0, Resistor_SMD:R_0805_2012Metric, F.Cu at (24.5, -61.9)
- added R1404: DNP, Resistor_SMD:R_0805_2012Metric, F.Cu at (20.1, -59.0)
- added R1405: 0, Resistor_SMD:R_0805_2012Metric, F.Cu at (24.5, -59.0)
- added R1406: DNP, Resistor_SMD:R_0805_2012Metric, F.Cu at (15.6, -56.0)
- added R1407: DNP, Resistor_SMD:R_0805_2012Metric, F.Cu at (20.1, -56.0)
- added R1408: 0, Resistor_SMD:R_0805_2012Metric, F.Cu at (15.6, -53.1)
- added R606: 200, Resistor_SMD:R_0805_2012Metric, F.Cu at (111.2, -60.9)
- added R607: 27, Resistor_SMD:R_0805_2012Metric, F.Cu at (120.3, -73.3)
- added R608: 200, Resistor_SMD:R_0805_2012Metric, F.Cu at (111.2, -58.0)
- added R609: 24, Resistor_SMD:R_0805_2012Metric, F.Cu at (106.8, -55.6)
- added R610: 24, Resistor_SMD:R_0805_2012Metric, F.Cu at (112.4, -63.9)
- added R611: 220, Resistor_SMD:R_0805_2012Metric, F.Cu at (102.3, -49.6)
- added R612: 220, Resistor_SMD:R_0805_2012Metric, F.Cu at (116.9, -66.9)
- added R613: 100, Resistor_SMD:R_0805_2012Metric, F.Cu at (125.9, -76.3)
- added R614: 100, Resistor_SMD:R_0805_2012Metric, F.Cu at (116.9, -64.0)
- added RN1401: 4x82R, Resistor_SMD:R_Array_Convex_4x0603, F.Cu at (23.8, -68.8)
- added RN1402: 4x82R, Resistor_SMD:R_Array_Convex_4x0603, F.Cu at (28.0, -68.8)
- added RN1403: 4x82R, Resistor_SMD:R_Array_Convex_4x0603, F.Cu at (15.5, -68.8)
- added RN1404: 4x82R, Resistor_SMD:R_Array_Convex_4x0603, F.Cu at (19.7, -68.8)
- added TP101: TestPoint, TestPoint:TestPoint_Bridge_Pitch5.08mm_Drill1.3mm, F.Cu at (148.1, 126.0)
- added TP102: TestPoint, TestPoint:TestPoint_Bridge_Pitch5.08mm_Drill1.3mm, F.Cu at (148.1, 121.3)
- added TP1201: TestPoint, TestPoint:TestPoint_THTPad_D1.0mm_Drill0.5mm, F.Cu at (-35.3, 14.5)
- added TP1202: TestPoint, TestPoint:TestPoint_THTPad_D1.0mm_Drill0.5mm, F.Cu at (-33.9, 11.5)
- added TP1203: TestPoint, TestPoint:TestPoint_THTPad_D1.0mm_Drill0.5mm, F.Cu at (-33.4, 8.42)
- added TP1204: TestPoint, TestPoint:TestPoint_THTPad_D1.0mm_Drill0.5mm, F.Cu at (-42.1, 21.7)
- added TP1205: TestPoint, TestPoint:TestPoint_THTPad_D1.0mm_Drill0.5mm, F.Cu at (-33.4, 5.37)
- added TP1206: TestPoint, TestPoint:TestPoint_THTPad_D1.0mm_Drill0.5mm, F.Cu at (-45.2, 22.5)
- added TP1207: TestPoint, TestPoint:TestPoint_THTPad_D1.0mm_Drill0.5mm, F.Cu at (-54.9, 33.0)
- added TP1208: TestPoint, TestPoint:TestPoint_THTPad_D1.0mm_Drill0.5mm, F.Cu at (-45.2, 25.5)
- added TP602: TestPoint, TestPoint:TestPoint_THTPad_D1.0mm_Drill0.5mm, F.Cu at (106.1, -52.6)
- added U1101: 74LVC2GU04, Package_TO_SOT_SMD:SOT-23-6, F.Cu at (85.8, -31.2)
- added U1102: 74LVC2G04, Package_TO_SOT_SMD:SOT-23-6, F.Cu at (90.5, -38.4)
- added U1201: TL431AFDT, Package_TO_SOT_SMD:SOT-23, F.Cu at (-41.8, 6.07)
- added U1202: TL431AFDT, Package_TO_SOT_SMD:SOT-23, F.Cu at (-59.4, 22.4)
- added U1203: TL431AFDT, Package_TO_SOT_SMD:SOT-23, F.Cu at (-67.7, 32.9)
- added U1204: MCP1824T-330, Package_TO_SOT_SMD:SOT-223-6, F.Cu at (-70.3, 16.2)
- added U1205: NCV8164ASN120T1G, Package_TO_SOT_SMD:SOT-23-5, F.Cu at (-51.3, 12.8)
- added U1206: MCP1824T-330, Package_TO_SOT_SMD:SOT-223-6, F.Cu at (-70.3, 7.97)
- added U1207: NCV8164ASN250T1G, Package_TO_SOT_SMD:SOT-23-5, F.Cu at (-72.7, 31.8)
- added U1208: NCV8164ASN330T1G, Package_TO_SOT_SMD:SOT-23-5, F.Cu at (-67.0, 28.4)
- added U1301: AT93C56, Package_SO:TSSOP-8_4.4x3mm_P0.65mm, F.Cu at (182.8, 119.2)
- added U1302: FT2232HL, Package_QFP:LQFP-64_10x10mm_P0.5mm, F.Cu at (215.3, 87.6)
- added U1401: 74AVC4T245PW, Package_SO:TSSOP-16_4.4x5mm_P0.65mm, F.Cu at (17.8, -74.5)
- added U1402: 74AVC4T245PW, Package_SO:TSSOP-16_4.4x5mm_P0.65mm, F.Cu at (26.6, -74.5)
- added U202: W25Q16JV, Package_SO:SOIC-8_5.23x5.23mm_P1.27mm, F.Cu at (-70.1, -5.53)
- added U203: IS61WV25616FBLL-10TLI, Package_SO:TSOP-II-44_10.16x18.41mm_P0.8mm, F.Cu at (196.8, 48.4)
- added X901: TXEAADSANF-20.0, Crystal:Crystal_SMD_3225-4Pin_3.2x2.5mm_HandSoldering, F.Cu at (-5.17, -26.5)
- added X902: DOT050V-020.0M, custom-footprints:ConnorWinfield_DOT050, F.Cu at (-14.2, -25.1)
- added Y1301: 12MHz CL=18p, Crystal:Crystal_SMD_3225-4Pin_3.2x2.5mm_HandSoldering, F.Cu at (195.5, 104.7)
- C1001: value 27p -> 4.7u
- C1002: value 27p -> 100n
- C1003, C903: value 4.7u -> 100n
- C201: value 3.3n -> 4.7u
- C203: value 8.2n -> 4.7u
- C204, C210, C304, C404, C504, C901: value 10n -> 100n
- C205: value 8.2n -> 1u
- C207: value 3.3n -> 100n
- C211, C212, C213, C214: value 1.5n -> 100n
- C301, C401, C501: value 3.3n -> 1u
- C303, C403, C503: value 8.2n -> 6.8n
- C305, C405, C505: value 8.2n -> 100n; footprint Capacitor_SMD:C_0805_2012Metric -> Capacitor_SMD:C_1206_3216Metric
- C306, C406, C506, C606: footprint Capacitor_SMD:C_0805_2012Metric -> Capacitor_SMD:C_1206_3216Metric
- C307, C407, C507: value 3.3n -> 10n
- C308, C309, C408, C409, C508, C509, C608, C609, C610, C611: value 100n -> 1.5n
- C310, C410, C510: value 10n -> 1.5n
- C601: value 100n -> 1u
- C605: value 300p -> 100n; footprint Capacitor_SMD:C_0805_2012Metric -> Capacitor_SMD:C_1206_3216Metric
- C607, C902: value 100n -> 10n
- C701, C702: value 100n -> 10u; footprint Capacitor_SMD:C_0805_2012Metric -> Capacitor_SMD:CP_Elec_4x5.8
- C801: value 1n -> 10u; footprint Capacitor_SMD:C_0805_2012Metric -> Capacitor_SMD:CP_Elec_4x5.8
- C802: value 10n -> 10u; footprint Capacitor_SMD:C_0805_2012Metric -> Capacitor_SMD:CP_Elec_4x5.8
- C803: value 100n/U2J -> 100n
- C805: value 100n -> 4.7u
- C904: value 1u -> 100n; footprint Capacitor_SMD:C_0805_2012Metric -> Capacitor_SMD:C_1206_3216Metric
- C908, C909: value 1u -> 100n
- C911: value 4.7u -> 1n
- C912: value 1u -> 10n
- D101: value IN1:R,G -> WP130WCP/2EGW; footprint LED_THT:LED_D3.0mm-3 -> custom-footprints:WP130WCP
- D102: value IN3:R,G -> WP130WCP/2EGW; footprint LED_THT:LED_D3.0mm-3 -> custom-footprints:WP130WCP
- D103: value STATUS:R,G -> WP130WCP/2EGW; footprint LED_THT:LED_D3.0mm-3 -> custom-footprints:WP130WCP
- J101: value USB_B -> IN1; footprint Connector_USB:USB_B_Lumberg_2411_02_Horizontal -> custom-footprints:SMA_Superbat_S01-ROPT4-11BS00
- R1001: value 5.1k -> 75
- R1002: value 10k -> 120
- R102, R103, R104, R105, R106, R107, R110, R111: value 1k -> 220
- R108, R109: value 10k -> 220
- R201: value 49.9 -> 220
- R202: value 0 -> 10k
- R203, R204: value 3.3k -> 10k
- R205: value 49.9 -> 10k
- R206: value 62 -> 10k
- R207: value 200 -> 100
- R208: value 27 -> 100
- R301, R401, R501: value 49.9 -> 0
- R302, R402, R502: value 0 -> 49.9
- R303, R304, R403, R404, R503, R504: value 3.3k -> 1k
- R305, R405, R505: value 49.9 -> 62
- R306, R406, R506: value 62 -> 200
- R307, R407, R507: value 200 -> 27
- R308, R408, R508: value 27 -> 200
- R309, R409, R509: value 200 -> 24
- R311, R411, R511: value 24 -> 220
- R313, R413, R513: value 220 -> 100
- R601: value 10k -> 0
- R602: value 100k -> 49.9
- R603: value 49.9 -> 1k
- R604: value 10k -> 1k
- R605: value 100k -> 62
- R901: value 100k -> 10k
- R902: value 5.1k -> 49.9
- R903: value 10k -> 2.4k
- R905: value 10k -> 100k
- U1001: value AT93C56 -> 74LVC1G157; footprint Package_SO:SOIC-8_3.9x4.9mm_P1.27mm -> Package_TO_SOT_SMD:SOT-23-6
- U1002: value FT2232HL -> 74LVC2G04; footprint Package_QFP:LQFP-64_10x10mm_P0.5mm -> Package_TO_SOT_SMD:SOT-23-6
- U201: value THS4521ID -> ICE40HX4K; footprint Package_SO:SOIC-8_3.9x4.9mm_P1.27mm -> Package_QFP:TQFP-144_20x20mm_P0.5mm
- U601: value DAC8551 -> THS4521ID; footprint Package_SO:VSSOP-8_3.0x3.0mm_P0.65mm -> Package_SO:SOIC-8_3.9x4.9mm_P1.27mm
- U701: value 74LVC1G157 -> AD7357xRU; footprint Package_TO_SOT_SMD:SOT-23-6 -> Package_SO:TSSOP-16_4.4x5mm_P0.65mm
- U801: value 74LVC2GU04 -> AD7357xRU; footprint Package_TO_SOT_SMD:SOT-23-6 -> Package_SO:TSSOP-16_4.4x5mm_P0.65mm
- U901: value MCP1825T-330 -> DAC8551; footprint Package_TO_SOT_SMD:SOT-223-6 -> Package_SO:VSSOP-8_3.0x3.0mm_P0.65mm
- U902: value NCV8164ASN120T1G -> MCP1501-33xSN; footprint Package_TO_SOT_SMD:SOT-23-5 -> Package_SO:SOIC-8_3.9x4.9mm_P1.27mm
- U903: value MCP1825T-330 -> NCS325; footprint Package_TO_SOT_SMD:SOT-223-6 -> Package_TO_SOT_SMD:SOT-23-5
- U904: value NCV8164ASN250T1G -> 74LVC2GU04; footprint Package_TO_SOT_SMD:SOT-23-5 -> Package_TO_SOT_SMD:SOT-23-6
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Connections:
- C1001 pad 1: Net-(C1001-Pad1) -> AGND
- C1001 pad 2: AGND -> /Clock Output/VDD_3V3
- C1002 pad 1: Net-(C1002-Pad1) -> AGND
- C1002 pad 2: AGND -> /Clock Output/VDD_3V3
- C1003 pad 1: /FTDI/FT_+1V8 -> Net-(C1003-Pad1)
- C1003 pad 2: AGND -> Net-(C1003-Pad2)
- C201 pad 1: /Input Amplifier 2/IN -> +3.3VD
- C201 pad 2: Net-(C201-Pad2) -> AGND
- C203 pad 1: Net-(C203-Pad1) -> +1.2VD
- C204 pad 1: Net-(C204-Pad1) -> +3.3VD
- C205 pad 1: Net-(C205-Pad1) -> +1.2VD
- C206 pad 1: /Input Amplifier 2/VOCM -> +3.3VD
- C206 pad 2: GNDA -> AGND
- C207 pad 1: Net-(C207-Pad1) -> +1.2VD
- C207 pad 2: Net-(C207-Pad2) -> AGND
- C208 pad 1: Net-(C207-Pad1) -> +3.3VD
- C208 pad 2: Net-(C208-Pad2) -> AGND
- C209 pad 1: AGND -> +1.2VD
- C209 pad 2: Net-(C209-Pad2) -> AGND
- C210 pad 1: Net-(C210-Pad1) -> +3.3VD
- C210 pad 2: Net-(C210-Pad2) -> AGND
- C211 pad 1: Net-(C211-Pad1) -> +1.2VD
- C211 pad 2: Net-(C211-Pad2) -> AGND
- C212 pad 1: Net-(C212-Pad1) -> +3.3VD
- C212 pad 2: Net-(C212-Pad2) -> AGND
- C213 pad 1: /Input Amplifier 2/OUT- -> +1.2VD
- C214 pad 1: /Input Amplifier 2/OUT+ -> +3.3VD
- C301 pad 1: /Input Amplifier 3/IN -> /Input Amplifier 1/VS+
- C301 pad 2: Net-(C301-Pad2) -> AGND
- C304 pad 1: Net-(C304-Pad1) -> /Input Amplifier 1/VOCM
- C305 pad 1: Net-(C305-Pad1) -> Net-(C303-Pad1)
- C305 pad 2: AGND -> Net-(C305-Pad2)
- C306 pad 1: /Input Amplifier 3/VOCM -> AGND
- C306 pad 2: GNDA -> Net-(C306-Pad2)
- C308 pad 1: Net-(C307-Pad1) -> Net-(C308-Pad1)
- C309 pad 1: AGND -> Net-(C309-Pad1)
- C310 pad 1: Net-(C310-Pad1) -> /ADC1/INA+
- C310 pad 2: Net-(C310-Pad2) -> AGND
- C311 pad 1: Net-(C311-Pad1) -> /ADC1/INA-
- C311 pad 2: Net-(C311-Pad2) -> AGND
- C401 pad 1: /Input Amplifier 1/IN -> /Input Amplifier 2/VS+
- C401 pad 2: Net-(C401-Pad2) -> AGND
- C404 pad 1: Net-(C404-Pad1) -> /Input Amplifier 2/VOCM
- C405 pad 1: Net-(C405-Pad1) -> Net-(C403-Pad1)
- C405 pad 2: AGND -> Net-(C405-Pad2)
- C406 pad 1: /Input Amplifier 1/VOCM -> AGND
- C406 pad 2: GNDA -> Net-(C406-Pad2)
- C408 pad 1: Net-(C407-Pad1) -> Net-(C408-Pad1)
- C409 pad 1: AGND -> Net-(C409-Pad1)
- C410 pad 1: Net-(C410-Pad1) -> /ADC1/INB-
- C410 pad 2: Net-(C410-Pad2) -> AGND
- C411 pad 1: Net-(C411-Pad1) -> /ADC1/INB+
- C411 pad 2: Net-(C411-Pad2) -> AGND
- C501 pad 1: /Input Amplifier 4/IN -> /Input Amplifier 3/VS+
- C501 pad 2: Net-(C501-Pad2) -> AGND
- C504 pad 1: Net-(C504-Pad1) -> /Input Amplifier 3/VOCM
- C505 pad 1: Net-(C505-Pad1) -> Net-(C503-Pad1)
- C505 pad 2: AGND -> Net-(C505-Pad2)
- C506 pad 1: /Input Amplifier 4/VOCM -> AGND
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Routing:
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Other:
- board outline added: 162 x 120 mm
- board text added: "Board: 162x120mm, for Hammond 1455P1601 case + screw holes for out-of-case mounting"
- board text added: "KEEPOUT - EXTRUSION"

Commit message: PCB: wip
Parts:
- removed H105: MountingHole_Pad, MountingHole:MountingHole_3.2mm_M3_Pad
- removed the R301 at (140.8, 82.4)
- removed the R303 at (122.8, 97.1)
- removed the R304 at (139.6, 85.3)
- removed R412, R512, R612: 220, Resistor_SMD:R_0805_2012Metric
- removed R413, R414, R513, R514, R613, R614: 100, Resistor_SMD:R_0805_2012Metric
- added C1315: 100n, Capacitor_SMD:C_0805_2012Metric, F.Cu at (208.8, 114.8)
- added R101: 1k, Resistor_SMD:R_0805_2012Metric, F.Cu at (104.8, 22.2)
- added R102: 1k, Resistor_SMD:R_0805_2012Metric, F.Cu at (100.4, 22.2)
- C1305: renamed from C1306; moved to B.Cu
- C1306: renamed from C1305; moved to B.Cu
- C1307: renamed from C1310; moved to B.Cu
- C1308: renamed from C1307; moved to B.Cu
- C1311: renamed from C1314; moved to B.Cu
- C1312: renamed from C1311; moved to B.Cu
- C1313: renamed from C1312; moved to B.Cu
- C1314: renamed from C1313; moved to B.Cu
- C219, C223, C301, C304, C401, C404, C501, C504, C601, C604, D1301, R1308: moved to B.Cu
- C220, C222, C701, C702, C801, C802: footprint Capacitor_SMD:CP_Elec_4x5.8 -> Capacitor_Tantalum_SMD:CP_EIA-2012-15_AVX-P
- R401, R501, R601: value 0 -> 49.9
- R402, R502, R602: value 49.9 -> 62
- R403, R503, R603: value 1k -> 200
- R404, R504, R604: value 1k -> 27
- R405, R505, R605: value 62 -> 200
- R406, R506, R606: value 200 -> 24
- R407, R507, R607: value 27 -> 24
- R408, R508, R608: value 200 -> 220
- R409, R509, R609: value 24 -> 220
- R410, R510, R610: value 24 -> 100
- R411, R511, R611: value 220 -> 100
- moved C203 401.6 mm to (348.0, 104.3)
- moved C204 401.6 mm to (347.8, 111.5)
- moved C205 401.6 mm to (334.5, 130.3)
- moved C206 401.6 mm to (347.8, 117.5)
- moved C208 401.6 mm to (345.7, 123.5)
- moved C210 401.6 mm to (334.5, 133.3)
- moved C212 401.6 mm to (330.0, 133.1)
- moved C213 401.6 mm to (348.0, 107.3)
- moved C214 401.6 mm to (347.8, 114.5)
- moved C215 401.6 mm to (330.0, 130.1)
- moved C220 401.6 mm to (316.7, 130.1)
- moved R201 401.6 mm to (304.7, 135.4)
- moved R202 401.6 mm to (345.7, 126.5)
- moved R203 401.6 mm to (350.2, 123.5)
- moved R204 401.6 mm to (343.4, 133.2)
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- renumbered C1304 to C1303, C1303 to C1304, C1308 to C1309, C1309 to C1310, R101 to R103, R102 to R104, R103 to R105, R104 to R106, R105 to R107, R106 to R108, R107 to R109, R108 to R110, R109 to R111, R110 to R112, R111 to R113, R302 to R301, R305 to R302, R306 to R303, R307 to R304, R308 to R305, R309 to R306, R310 to R307, R311 to R308, R312 to R309, R313 to R310, R314 to R311, TP102 to TP101, TP101 to TP102
Connections:
- net /FTDI/USB_DM renamed /FTDI/USB_D-
- net /FTDI/USB_DP renamed /FTDI/USB_D+
- net Net-(R1303-Pad2) renamed /FTDI/USB_DR-
- net Net-(R1304-Pad2) renamed /FTDI/USB_DR+
- C301 pad 1: /Input Amplifier 1/VS+ -> +3.3VA
- C401 pad 1: /Input Amplifier 2/VS+ -> +3.3VA
- C404 pad 1: /Input Amplifier 2/VOCM -> /Input Amplifier 1/VOCM
- C501 pad 1: /Input Amplifier 3/VS+ -> +3.3VA
- C504 pad 1: /Input Amplifier 3/VOCM -> /Input Amplifier 1/VOCM
- C601 pad 1: /Input Amplifier 4/VS+ -> +3.3VA
- C604 pad 1: /Input Amplifier 4/VOCM -> /Input Amplifier 1/VOCM
- D303 pad 1: /Input Amplifier 1/VS+ -> +3.3VA
- D403 pad 1: /Input Amplifier 2/VS+ -> +3.3VA
- D503 pad 1: /Input Amplifier 3/VS+ -> +3.3VA
- D603 pad 1: /Input Amplifier 4/VS+ -> +3.3VA
- R1311 pad 2: /FTDI/FT_+3V3 -> /FTDI/FT_3V3
- R401 pad 1: /Input Amplifier 2/VS+ -> Net-(C402-Pad2)
- R401 pad 2: +3.3VA -> AGND
- R402 pad 1: Net-(C402-Pad2) -> AGND
- R402 pad 2: AGND -> Net-(C403-Pad1)
- R403 pad 1: /Input Amplifier 2/VOCM -> Net-(C405-Pad2)
- R403 pad 2: +2.5VA -> Net-(C407-Pad2)
- R404 pad 1: AGND -> Net-(C406-Pad2)
- R404 pad 2: /Input Amplifier 2/VOCM -> Net-(R404-Pad2)
- R405 pad 1: AGND -> Net-(R404-Pad2)
- R405 pad 2: Net-(C403-Pad1) -> Net-(C407-Pad1)
- R406 pad 1: Net-(C405-Pad2) -> Net-(C407-Pad2)
- R406 pad 2: Net-(C407-Pad2) -> Net-(C408-Pad2)
- R407 pad 1: Net-(C406-Pad2) -> Net-(C407-Pad1)
- R407 pad 2: Net-(R407-Pad2) -> Net-(C409-Pad2)
- R408 pad 1: Net-(R407-Pad2) -> Net-(C407-Pad2)
- R408 pad 2: Net-(C407-Pad1) -> Net-(C408-Pad1)
- R409 pad 1: Net-(C407-Pad2) -> Net-(C407-Pad1)
- R409 pad 2: Net-(C408-Pad2) -> Net-(C409-Pad1)
- R410 pad 1: Net-(C407-Pad1) -> Net-(C408-Pad1)
- R410 pad 2: Net-(C409-Pad2) -> /ADC1/INB-
- R411 pad 1: Net-(C407-Pad2) -> Net-(C409-Pad1)
- R411 pad 2: Net-(C408-Pad1) -> /ADC1/INB+
- R501 pad 1: /Input Amplifier 3/VS+ -> Net-(C502-Pad2)
- R501 pad 2: +3.3VA -> AGND
- R502 pad 1: Net-(C502-Pad2) -> AGND
- R502 pad 2: AGND -> Net-(C503-Pad1)
- R503 pad 1: /Input Amplifier 3/VOCM -> Net-(C505-Pad2)
- R503 pad 2: +2.5VA -> Net-(C507-Pad2)
- R504 pad 1: AGND -> Net-(C506-Pad2)
- R504 pad 2: /Input Amplifier 3/VOCM -> Net-(R504-Pad2)
- R505 pad 1: AGND -> Net-(R504-Pad2)
- R505 pad 2: Net-(C503-Pad1) -> Net-(C507-Pad1)
- R506 pad 1: Net-(C505-Pad2) -> Net-(C507-Pad2)
- R506 pad 2: Net-(C507-Pad2) -> Net-(C508-Pad2)
- R507 pad 1: Net-(C506-Pad2) -> Net-(C507-Pad1)
- R507 pad 2: Net-(R507-Pad2) -> Net-(C509-Pad2)
- R508 pad 1: Net-(R507-Pad2) -> Net-(C507-Pad2)
- R508 pad 2: Net-(C507-Pad1) -> Net-(C508-Pad1)
- R509 pad 1: Net-(C507-Pad2) -> Net-(C507-Pad1)
- R509 pad 2: Net-(C508-Pad2) -> Net-(C509-Pad1)
- R510 pad 1: Net-(C507-Pad1) -> Net-(C508-Pad1)
- R510 pad 2: Net-(C509-Pad2) -> /ADC2/INA+
- R511 pad 1: Net-(C507-Pad2) -> Net-(C509-Pad1)
- R511 pad 2: Net-(C508-Pad1) -> /ADC2/INA-
- R601 pad 1: /Input Amplifier 4/VS+ -> Net-(C602-Pad2)
- R601 pad 2: +3.3VA -> AGND
- R602 pad 1: Net-(C602-Pad2) -> AGND
- R602 pad 2: AGND -> Net-(C603-Pad1)
- R603 pad 1: /Input Amplifier 4/VOCM -> Net-(C605-Pad2)
- R603 pad 2: +2.5VA -> Net-(C607-Pad2)
- R604 pad 1: AGND -> Net-(C606-Pad2)
- R604 pad 2: /Input Amplifier 4/VOCM -> Net-(R604-Pad2)
- R605 pad 1: AGND -> Net-(R604-Pad2)
- R605 pad 2: Net-(C603-Pad1) -> Net-(C607-Pad1)
- R606 pad 1: Net-(C605-Pad2) -> Net-(C607-Pad2)
- R606 pad 2: Net-(C607-Pad2) -> Net-(C608-Pad2)
- R607 pad 1: Net-(C606-Pad2) -> Net-(C607-Pad1)
- R607 pad 2: Net-(R607-Pad2) -> Net-(C609-Pad2)
- R608 pad 1: Net-(R607-Pad2) -> Net-(C607-Pad2)
- R608 pad 2: Net-(C607-Pad1) -> Net-(C608-Pad1)
- R609 pad 1: Net-(C607-Pad2) -> Net-(C607-Pad1)
- R609 pad 2: Net-(C608-Pad2) -> Net-(C609-Pad1)
- R610 pad 1: Net-(C607-Pad1) -> Net-(C608-Pad1)
- R610 pad 2: Net-(C609-Pad2) -> /ADC2/INB-
- R611 pad 1: Net-(C607-Pad2) -> Net-(C609-Pad1)
- R611 pad 2: Net-(C608-Pad1) -> /ADC2/INB+
- U201 pad 25: /FPGA/LED.IN_G1 -> /FPGA/LED.IN_R2
- U201 pad 26: /FPGA/LED.IN_R2 -> /FPGA/LED.IN_G2
- U201 pad 28: /FPGA/LED.IN_G2 -> /FPGA/LED.IN_G1
- U201 pad 31: /FPGA/LED.IN_G3 -> /FPGA/LED.IN_R4
- U201 pad 32: /FPGA/LED.IN_R4 -> /FPGA/LED.IN_G4
- U201 pad 33: /FPGA/LED.IN_G4 -> /FPGA/LED.IN_G3
- U301 pad 3: /Input Amplifier 1/VS+ -> +3.3VA
- U401 pad 2: /Input Amplifier 2/VOCM -> /Input Amplifier 1/VOCM
- U401 pad 3: /Input Amplifier 2/VS+ -> +3.3VA
- U501 pad 2: /Input Amplifier 3/VOCM -> /Input Amplifier 1/VOCM
- U501 pad 3: /Input Amplifier 3/VS+ -> +3.3VA
- U601 pad 2: /Input Amplifier 4/VOCM -> /Input Amplifier 1/VOCM
- U601 pad 3: /Input Amplifier 4/VS+ -> +3.3VA
Routing:
- net +3.3VA: track 0.00 -> 100.4 mm, vias 0 -> 4
- net /Input Amplifier 1/VOCM: track 0.00 -> 72.2 mm, vias 0 -> 4
- net /FTDI/FT_3V3: track 0.00 -> 67.6 mm, vias 0 -> 6
- net AGND: track 0.00 -> 64.1 mm, vias 0 -> 51
- net Net-(D102-Pad4): track 0.00 -> 58.2 mm
- net Net-(D102-Pad6): track 0.00 -> 57.7 mm
- net Net-(D103-Pad4): track 0.00 -> 57.2 mm
- net Net-(D103-Pad6): track 0.00 -> 56.7 mm
- net Net-(D102-Pad1): track 0.00 -> 55.1 mm
- net Net-(D102-Pad3): track 0.00 -> 54.6 mm
- net Net-(D103-Pad1): track 0.00 -> 54.1 mm
- net Net-(D103-Pad3): track 0.00 -> 53.6 mm
- net /FPGA/LED.IN_G3: track 0.00 -> 45.5 mm
- net /ADC1/ADC.SCK: track 0.00 -> 44.1 mm
- net /FPGA/LED.IN_G1: track 0.00 -> 43.4 mm
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- added copper zone on B.Cu, net AGND
- added copper zone on F.Cu, net AGND
