File: lwdo-sdr.kicad_pcb (KiCad board)
At the start: 2 copper layers, 162 x 120 mm, 367 parts, among them J101 IN1, J102 IN2, J103 IN3, J104 IN4, J105 USB_B, J106 CLK_OUT, J107 REF_IN, J1401 Conn_02x10_Odd_Even, Q1201 NX7002AK, Q1202 PMN48XP, U1001 74LVC1G157, U1002 74LVC2G04, U1101 74LVC2GU04, U1102 74LVC2G04, U1201 TL431AFDT, U1202 TL431AFDT, U1203 TL431AFDT, U1204 MCP1824T-330, U1205 NCV8164ASN120T1G, U1206 MCP1824T-330, U1207 NCV8164ASN250T1G, U1208 NCV8164ASN330T1G, U1301 AT93C56, U1302 FT2232HL, U1401 74AVC4T245PW, U1402 74AVC4T245PW, U201 ICE40HX4K, U202 W25Q16JV, U203 IS61WV25616FBLL-10TLI, U301 THS4521ID, U401 THS4521ID, U501 THS4521ID, U601 THS4521ID, U701 AD7357xRU, U801 AD7357xRU, U901 DAC8551, U902 MCP1501-33xSN, U903 NCS325, U904 74LVC2GU04, U905 74LVC2G04, X901 TXEAADSANF-20.0, X902 DOT050V-020.0M, Y1301 12MHz CL=18p

Commit message: Reconnect some things to simplify PCB routing
Parts:
- removed C1406: 100n, Capacitor_SMD:C_0805_2012Metric
- added C901: 100n, Capacitor_SMD:C_0805_2012Metric, F.Cu at (168.1, 120.7)
- added H105: MountingHole_Pad, MountingHole:MountingHole_3.2mm_M3_Pad, F.Cu at (113.5, -23.8)
- C1001, C1002, C1104, C1105: moved to B.Cu
- C902: renamed from C901; moved to B.Cu
- C910: renamed from C908; moved to B.Cu
- C911: renamed from C909; moved to B.Cu
- moved C913 256.2 mm to (198.2, 138.4), turned to 90 degrees
- moved U904 256.0 mm to (199.3, 133.3), turned to 90 degrees
- moved X902 255.2 mm to (186.6, 132.5)
- moved J1401 254.6 mm to (150.6, 138.4), turned to -90 degrees
- moved R905 253.8 mm to (200.5, 138.4), turned to 90 degrees
- moved U905 253.0 mm to (199.3, 127.0), turned to 90 degrees
- moved C910 251.0 mm to (199.3, 133.3), turned to 90 degrees
- moved U1002 249.1 mm to (218.3, 133.9)
- moved D1001 249.1 mm to (218.3, 137.0)
- moved JP1001 249.1 mm to (222.9, 120.7), turned to 180 degrees
- moved X901 249.1 mm to (186.6, 132.5), turned to -90 degrees
- moved D1003 248.9 mm to (234.4, 119.0), turned to 90 degrees
- moved C911 247.7 mm to (199.3, 127.0), turned to 90 degrees
- moved C912 247.6 mm to (194.9, 135.0), turned to 180 degrees
- moved R904 247.3 mm to (196.0, 138.4), turned to -90 degrees
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- renumbered C910 to C903, C902 to C904, C903 to C905, C904 to C906, C905 to C907, C906 to C908, C907 to C909, C911 to C912, C912 to C913
Connections:
- C1003 pad 2: Net-(C1003-Pad2) -> /Clock Output/OUT
- C1102 pad 1: Net-(C1102-Pad1) -> /Reference Clock Input/IN
- C1102 pad 2: Net-(C1102-Pad2) -> Net-(R1102-Pad2)
- C903 pad 2: +3.3VD -> +3.3VA
- D1001 pad 2: Net-(C1003-Pad1) -> Net-(D1001-Pad2)
- D1002 pad 1: Net-(C1003-Pad1) -> Net-(D1001-Pad2)
- D1003 pad 1: AGND -> /Clock Output/OUT
- D1003 pad 2: /Clock Output/OUT -> AGND
- D1102 pad 1: Net-(C1102-Pad2) -> Net-(D1102-Pad1)
- D1103 pad 2: Net-(C1102-Pad2) -> Net-(D1102-Pad1)
- J1401 pad 11: /Extension Connector/IO4 -> /Extension Connector/EXT_IO4
- J1401 pad 13: /Extension Connector/IO5 -> /Extension Connector/EXT_IO5
- J1401 pad 15: /Extension Connector/IO6 -> /Extension Connector/EXT_IO6
- J1401 pad 17: /Extension Connector/IO7 -> /Extension Connector/EXT_IO7
- J1401 pad 19: /Extension Connector/IO8 -> /Extension Connector/EXT_IO8
- J1401 pad 5: /Extension Connector/IO1 -> /Extension Connector/EXT_IO1
- J1401 pad 7: /Extension Connector/IO2 -> /Extension Connector/EXT_IO2
- J1401 pad 9: /Extension Connector/IO3 -> /Extension Connector/EXT_IO3
- JP1001 pad 2: Net-(C1003-Pad2) -> /Clock Output/OUT
- JP1101 pad 1: Net-(C1102-Pad1) -> /Reference Clock Input/IN
- JP1101 pad 2: Net-(C1102-Pad2) -> Net-(R1102-Pad2)
- R1001 pad 1: /Clock Output/OUT -> Net-(C1003-Pad1)
- R1001 pad 2: Net-(C1003-Pad2) -> Net-(D1001-Pad2)
- R1102 pad 1: Net-(C1102-Pad1) -> Net-(D1102-Pad1)
- R1102 pad 2: /Reference Clock Input/IN -> Net-(R1102-Pad2)
- R1103 pad 1: Net-(C1102-Pad2) -> Net-(D1102-Pad1)
- RN1403 pad 5: /Extension Connector/IO4 -> /Extension Connector/EXT_IO4
- RN1403 pad 6: /Extension Connector/IO3 -> /Extension Connector/EXT_IO3
- RN1403 pad 7: /Extension Connector/IO2 -> /Extension Connector/EXT_IO2
- RN1403 pad 8: /Extension Connector/IO1 -> /Extension Connector/EXT_IO1
- RN1404 pad 5: /Extension Connector/IO8 -> /Extension Connector/EXT_IO8
- RN1404 pad 6: /Extension Connector/IO7 -> /Extension Connector/EXT_IO7
- RN1404 pad 7: /Extension Connector/IO6 -> /Extension Connector/EXT_IO6
- RN1404 pad 8: /Extension Connector/IO5 -> /Extension Connector/EXT_IO5
- U1002 pad 4: Net-(C1003-Pad1) -> Net-(D1001-Pad2)
- U1002 pad 6: Net-(C1003-Pad1) -> Net-(D1001-Pad2)
- U1101 pad 1: Net-(C1102-Pad2) -> Net-(R1104-Pad1)
- U1101 pad 3: Net-(R1104-Pad1) -> Net-(D1102-Pad1)
- U1101 pad 4: Net-(U1101-Pad4) -> Net-(R1104-Pad1)
- U1101 pad 6: Net-(R1104-Pad1) -> Net-(U1101-Pad6)
- U1102 pad 1: Net-(U1101-Pad4) -> Net-(U1102-Pad1)
- U1102 pad 3: Net-(U1102-Pad3) -> Net-(U1101-Pad6)
- U1102 pad 4: /FPGA/REF_CLK_IN -> Net-(U1102-Pad1)
- U1102 pad 6: Net-(U1102-Pad3) -> /FPGA/REF_CLK_IN
- U201 pad 56: /Clock Output/CLK0 -> /Clock Output/CLK1
- U201 pad 63: /FPGA/QSPI_IO2 -> /FPGA/QSPI_IO3
- U201 pad 64: /FPGA/QSPI_IO3 -> /FPGA/QSPI_IO2
- U901 pad 1: +3.3VD -> +3.3VA
- U905 pad 4: /Clock Output/CLK1 -> /Clock Output/CLK0
Routing:
- net Net-(D103-Pad3): track 53.6 -> 0.00 mm
- net /Extension Connector/DIR12: track 0.00 -> 51.9 mm
- net Net-(D103-Pad6): track 56.7 -> 5.49 mm
- net Net-(D103-Pad4): track 57.2 -> 7.67 mm
- net Net-(D103-Pad1): track 54.1 -> 5.13 mm
- net /Extension Connector/DIR34: track 0.00 -> 47.9 mm
- net Net-(D102-Pad3): track 54.6 -> 9.62 mm
- net Net-(D102-Pad6): track 57.7 -> 13.2 mm
- net Net-(D102-Pad4): track 58.2 -> 14.2 mm
- net Net-(D102-Pad1): track 55.1 -> 11.7 mm
- net /Extension Connector/DIR56: track 0.00 -> 41.2 mm
- net /Extension Connector/DIR78: track 0.00 -> 37.0 mm
- net /ADC1/INA+: track 35.4 -> 0.00 mm
- net /ADC1/INA-: track 34.1 -> 0.00 mm
- net /FPGA/LED.IN_R1: track 30.5 -> 58.3 mm
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- removed copper zone on F.Cu, net AGND

Commit message: PCB: WIP
Parts:
- C204, C206, C208, C210, C211, C212, C213, C214, C215, C220, C221, C222, R207, R208: moved to B.Cu
- moved C214 191.0 mm to (160.0, 79.4), turned to 180 degrees
- moved C206 189.1 mm to (166.8, 63.0), turned to 90 degrees
- moved R207 186.4 mm to (174.4, 64.5), turned to -90 degrees
- moved C215 179.2 mm to (161.5, 69.0), turned to 180 degrees
- moved C204 177.5 mm to (172.8, 81.3)
- moved C213 175.5 mm to (178.2, 63.0), turned to 90 degrees
- moved C208 171.9 mm to (182.8, 68.7)
- moved C203 165.7 mm to (193.3, 45.0)
- moved C210 162.7 mm to (182.8, 74.4)
- moved C205 162.2 mm to (193.3, 50.4)
- moved C212 157.3 mm to (180.7, 83.7), turned to 90 degrees
- moved C217 153.7 mm to (206.0, 42.5)
- moved C216 153.5 mm to (206.1, 45.7)
- moved R208 149.3 mm to (169.9, 81.4), turned to 90 degrees
- moved C201 142.7 mm to (215.1, 52.8)
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Connections:
- U201 pad 61: /FPGA/FT_IO.IO1 -> /FPGA/QSPI_IO3
- U201 pad 62: /FPGA/FT_IO.IO2 -> /FPGA/QSPI_IO2
- U201 pad 63: /FPGA/QSPI_IO3 -> /FPGA/FT_IO.IO2
- U201 pad 64: /FPGA/QSPI_IO2 -> /FPGA/FT_IO.IO1
Routing:
- net +1.2VD: track 0.00 -> 48.2 mm, vias 0 -> 1
- net +3.3VD: track 57.7 -> 99.0 mm, vias 1 -> 8
- net /FPGA/FT_SPI.~{CS}: track 0.00 -> 32.8 mm, vias 0 -> 4
- net AGND: track 73.9 -> 102.1 mm, vias 39 -> 55
- net /FPGA/FT_SPI.MISO: track 2.32 -> 30.5 mm, vias 0 -> 2
- net /FPGA/FT_IO.IO2: track 1.98 -> 26.1 mm
- net /FPGA/FT_IO.IO1: track 2.34 -> 24.8 mm
- net Net-(JP201-Pad1): track 14.4 -> 36.5 mm, vias 0 -> 4
- net /FPGA/FT_SPI.MOSI: track 2.54 -> 24.1 mm, vias 0 -> 2
- net /FPGA/QSPI_IO3: track 0.00 -> 21.2 mm, vias 0 -> 2
- net /FPGA/FT_IO.CDONE: track 2.76 -> 23.5 mm
- net Net-(JP201-Pad4): track 5.98 -> 25.5 mm, vias 0 -> 4
- net /FPGA/FT_IO.~{CRESET}: track 3.18 -> 22.2 mm
- net /FPGA/FT_SPI.SCK: track 21.8 -> 33.5 mm, vias 0 -> 2
- net Net-(JP201-Pad2): track 0.00 -> 9.87 mm
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
Commit message: PCB: WIP
Parts:
- removed the D1203 at (-72.4, 27.9)
- removed D1204, D1206, D1207: SBR3U40S1F, Diode_SMD:D_SOD-123F
- removed JP1201: USB_PON, Connector_PinHeader_2.54mm:PinHeader_1x03_P2.54mm_Vertical
- added R1208: DNP, Resistor_SMD:R_0805_2012Metric, F.Cu at (206.1, 141.1)
- added R1209: 0, Resistor_SMD:R_0805_2012Metric, F.Cu at (206.1, 135.5)
- added R1211: DNP, Resistor_SMD:R_0805_2012Metric, F.Cu at (205.0, 138.3)
- added R1212: DNP, Resistor_SMD:R_0805_2012Metric, F.Cu at (203.8, 141.1)
- added R1213: 0, Resistor_SMD:R_0805_2012Metric, F.Cu at (203.8, 135.5)
- C207, C209: moved to B.Cu
- moved U1204 310.4 mm to (215.9, 136.3), turned to 90 degrees
- moved D1203 306.4 mm to (222.2, 142.2)
- moved C1211 302.0 mm to (217.8, 142.2), turned to 180 degrees
- moved Q1201 289.9 mm to (215.9, 128.9), turned to 180 degrees
- moved C1208 288.3 mm to (214.0, 142.2)
- moved TP1203 286.2 mm to (221.0, 139.7)
- moved R1210 284.7 mm to (210.4, 128.3), turned to 90 degrees
- moved C1209 275.7 mm to (208.3, 128.3), turned to -90 degrees
- moved TP1201 274.9 mm to (208.3, 142.0)
- moved C1203 255.9 mm to (168.5, 141.0), turned to -90 degrees
- moved FB1201 254.6 mm to (167.4, 138.0), turned to 180 degrees
- moved F1201 253.0 mm to (162.6, 138.4)
- moved C1201 252.5 mm to (166.2, 141.0), turned to -90 degrees
- moved D1201 252.0 mm to (162.6, 141.0), turned to 180 degrees
- moved C1205 251.6 mm to (170.8, 141.0), turned to -90 degrees
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- renumbered C1208 to C1207, C1207 to C1208, C1210 to C1209, C1211 to C1210, C1209 to C1211, D1205 to D1203, R1208 to R1210, R1209 to R1214, R1210 to R1215, R1211 to R1216, R1212 to R1217
Connections:
- net /FTDI/VBUS_CLEAN renamed /Power Supply/VBUS_CLEAN
- net /Power Supply/IN_VBUS renamed /Power Supply/VBUS
- net Net-(C1203-Pad1) renamed /Power Supply/5VEXT_CLEAN
- net Net-(C1207-Pad1) renamed /Power Supply/+5VFTDI
- Q1201 pad 3: Net-(JP1201-Pad1) -> Net-(Q1201-Pad3)
- R1210 pad 2: Net-(JP1201-Pad2) -> Net-(Q1201-Pad3)
Routing:
- net /Extension Connector/IO7: track 0.00 -> 44.4 mm
- net /Extension Connector/IO6: track 0.00 -> 44.2 mm
- net /Extension Connector/IO5: track 0.00 -> 44.1 mm
- net /Extension Connector/IO8: track 5.20 -> 47.5 mm
- net /Extension Connector/IO4: track 0.00 -> 41.8 mm
- net /Extension Connector/IO3: track 0.00 -> 41.7 mm
- net /Extension Connector/IO2: track 0.00 -> 41.6 mm
- net /Extension Connector/IO1: track 0.00 -> 41.5 mm
- net /ADC2/INB+: track 36.8 -> 0.00 mm
- net /ADC2/INB-: track 35.5 -> 0.00 mm
- net /FPGA/LED.IN_G3: track 51.9 -> 87.1 mm
- net /Extension Connector/OUT_5VEXT: track 0.00 -> 13.1 mm
- net /Extension Connector/EXT_IO8: track 12.9 -> 0.00 mm
- net +1.2VD: track 48.2 -> 58.4 mm, vias 1 -> 6
- net Net-(C1209-Pad1): track 0.00 -> 9.82 mm
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
Commit message: PCB: WIP - Power supply almost laid out
Parts:
- removed JP201: FLASH/CRAM, Connector_PinHeader_2.54mm:PinHeader_2x02_P2.54mm_Vertical
- removed JP202: FLASH/CRAM, Connector_PinHeader_2.54mm:PinHeader_1x02_P2.54mm_Vertical
- removed the R201 at (189.2, 100.3)
- C216, R1214, R1216, R1217: moved to B.Cu
- moved U1206 293.3 mm to (193.0, 137.2), turned to -90 degrees
- moved U1205 281.6 mm to (200.7, 138.4), turned to 90 degrees
- moved R1214 280.7 mm to (202.9, 141.5), turned to -90 degrees
- moved U1207 279.3 mm to (185.4, 138.4), turned to 90 degrees
- moved C1217 272.3 mm to (180.3, 135.0)
- moved C1210 271.7 mm to (175.3, 137.2), turned to 90 degrees
- moved U1203 271.0 mm to (185.4, 129.5), turned to 90 degrees
- moved C1214 270.8 mm to (200.7, 135.0)
- moved U1208 270.7 mm to (180.3, 138.4), turned to 90 degrees
- moved R1202 269.5 mm to (194.1, 125.9), turned to 90 degrees
- moved C1215 269.4 mm to (191.1, 131.3)
- moved C1212 268.8 mm to (194.9, 131.3), turned to 180 degrees
- moved C1213 266.5 mm to (177.9, 141.9), turned to 180 degrees
- moved C1216 265.2 mm to (185.4, 135.0)
- moved R1215 264.0 mm to (198.0, 132.1), turned to 90 degrees
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- renumbered R202 to R201, R203 to R202, R204 to R203, R205 to R204, R206 to R205, R207 to R206, R208 to R207
Connections:
- R201 pad 2: Net-(JP202-Pad2) -> /FPGA/FT_SPI.~{CS}
- U1302 pad 54: unconnected-(U1302-Pad54) -> Net-(R1311-Pad1)
- U201 pad 67: Net-(JP201-Pad1) -> /FPGA/FT_SPI.MOSI
- U201 pad 68: Net-(JP201-Pad4) -> /FPGA/FT_SPI.MISO
- U202 pad 1: Net-(JP202-Pad2) -> /FPGA/FT_SPI.~{CS}
- U202 pad 2: Net-(JP201-Pad4) -> /FPGA/FT_SPI.MISO
- U202 pad 5: Net-(JP201-Pad1) -> /FPGA/FT_SPI.MOSI
Routing:
- net /Power Supply/VBUS_CLEAN: track 1.82 -> 133.3 mm
- net /FTDI/~{PWREN}: track 6.61 -> 96.7 mm
- net /FTDI/FT_3V3: track 63.0 -> 152.9 mm, vias 4 -> 6
- net +5VMAIN: track 0.00 -> 65.9 mm, vias 0 -> 3
- net /Power Supply/5VEXT_CLEAN: track 2.10 -> 47.7 mm
- net Net-(JP201-Pad1): track 36.5 -> 0.00 mm, vias 4 -> 0
- net Net-(R1214-Pad1): track 0.00 -> 26.1 mm, vias 0 -> 1
- net Net-(JP201-Pad4): track 25.5 -> 0.00 mm, vias 4 -> 0
- net AGND: track 102.1 -> 120.7 mm, vias 55 -> 62
- net /FPGA/FT_SPI.MOSI: track 24.1 -> 38.5 mm, vias 2 -> 3
- net /Power Supply/+5VFTDI: track 6.61 -> 19.5 mm
- net Net-(R1215-Pad1): track 0.00 -> 12.5 mm
- net +3.3VD: track 102.6 -> 113.4 mm, vias 8 -> 9
- net Net-(JP201-Pad2): track 9.87 -> 0.00 mm
- net /Power Supply/VBUS: track 0.00 -> 9.16 mm
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
Commit message: PCB: WIP
Parts:
- removed the C907 at (165.6, 162.2)
- removed the X901 at (180.3, 110.7)
- added C909: 4.7u, Capacitor_SMD:C_0805_2012Metric, F.Cu at (190.1, 109.0)
- added R1105: 49.9, Resistor_SMD:R_0805_2012Metric, F.Cu at (204.0, 109.2)
- added R906: 49.9, Resistor_SMD:R_0805_2012Metric, F.Cu at (191.3, 101.9)
- C905: moved to B.Cu
- C907: renamed from C909; moved to B.Cu
- moved R201 192.6 mm to (182.8, 79.6), turned to -90 degrees
- moved R204 188.3 mm to (184.2, 76.7)
- moved R205 186.7 mm to (184.9, 79.6), turned to -90 degrees
- moved R202 183.1 mm to (189.5, 92.5), turned to 180 degrees
- moved R203 182.8 mm to (188.7, 89.7), turned to -90 degrees
- moved C907 55.0 mm to (184.5, 108.2)
- moved FB901 54.5 mm to (188.0, 105.4), turned to -90 degrees
- moved C905 50.5 mm to (184.5, 110.6)
- moved C903 22.5 mm to (159.6, 98.9)
- moved D1002 9.99 mm to (214.6, 122.4)
- moved R1001 9.68 mm to (221.1, 124.5), turned to 180 degrees
- moved C1209 9.65 mm to (212.0, 126.6), turned to 0 degrees
- moved JP1101 9.28 mm to (226.1, 109.2), turned to -90 degrees
- moved U1101 9.18 mm to (214.6, 109.2)
- moved C1104 8.81 mm to (214.2, 109.2)
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- renumbered X902 to X901
Connections:
- U1102 pad 6: /FPGA/REF_CLK_IN -> Net-(R1105-Pad1)
- U201 pad 55: /Clock Output/CLK_SEL -> /Clock Output/CLK1
- U201 pad 56: /Clock Output/CLK1 -> /Clock Output/CLK_SEL
- U905 pad 6: /FPGA/CLK_20MHZ -> Net-(R906-Pad1)
Routing:
- net /Clock Output/CLK_SEL: track 4.58 -> 70.9 mm
- net /Clock Output/CLK1: track 4.58 -> 70.3 mm
- net +3.3VD: track 113.4 -> 173.1 mm, vias 9 -> 13
- net /FPGA/REF_CLK_IN: track 5.19 -> 55.8 mm
- net /FPGA/CLK_20MHZ: track 4.30 -> 47.4 mm
- net +3.3VA: track 107.0 -> 144.9 mm, vias 4 -> 5
- net AGND: track 120.7 -> 154.6 mm, vias 62 -> 159
- net /Clock Output/CLK0: track 0.00 -> 24.4 mm
- net /Clock Output/OUT: track 0.00 -> 21.6 mm
- net /Reference Clock Input/IN: track 0.00 -> 20.6 mm
- net /FPGA/VCXO_DAC.SCK: track 0.74 -> 20.9 mm
- net /FPGA/VCXO_DAC.~{SYNC}: track 0.78 -> 20.9 mm
- net /FPGA/VCXO_DAC.DIN: track 1.20 -> 20.8 mm
- net Net-(D1001-Pad2): track 0.00 -> 16.4 mm
- net /Clock Output/VDD_3V3: track 0.00 -> 13.9 mm, vias 0 -> 2
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- added copper zone on F.Cu, net AGND
- added copper zone on F.Cu, net Net-(C1209-Pad1)
