File: power_supply.kicad_sch (KiCad schematic)
At the start: 59 parts, among them Q1201 NX7002AK, Q1202 PMN48XP, U1201 TL431AFDT, U1202 TL431AFDT, U1203 TL431AFDT, U1204 MCP1824T-330, U1205 NCV8164ASN120T1G, U1206 MCP1824T-330, U1207 NCV8164ASN250T1G, U1208 NCV8164ASN330T1G

Commit message: Update schematic: - Redesign of decoupling based on swcad modelling (predominantly use 1uf, no paralleled caps) - Reroute REF_CLK_IN, CLK_SEL net to different FPGA pins - Some net renaming - Ext conn: add decoupling to 3v3 output - Reassign references to all components PCB: routing almost finished
Parts:
- removed C1201: 100n, Capacitor_SMD:C_0805_2012Metric, symbol Device:C
- removed C1205: 4.7u, Capacitor_SMD:C_0805_2012Metric, symbol Device:C
- removed C1216, C1217: 1u, Capacitor_SMD:C_0805_2012Metric, symbol Device:C
- added C1209: 1u, Capacitor_SMD:C_0805_2012Metric, symbol Device:C
- added C1210: 4.7u, Capacitor_SMD:C_0805_2012Metric, symbol Device:C
- C1202, C1203, C1204: value 100n -> 1u; Mfr PN CL21B104KBFNNNE -> CL21B105KOFNNNG
- C1206: value 4.7u -> 1u; Mfr Murata -> Samsung; Mfr PN GRM21BR71C475ME51 -> CL21B105KOFNNNG
- C1211, C1212, C1213, C1214, C1215: value 1u -> 4.7u; Mfr Samsung -> Murata; Mfr PN CL21B105KOFNNNG -> GRM21BR71C475ME51
- renumbered C1208 to C1201, C1207 to C1205, C1209 to C1207, C1210 to C1208
Connections:
- net +5VFTDI: now also C1206.1; no longer C1201.1
- net 1V2D: now also C1212.1; no longer C1214.1
- net 2V5A: now also C1214.1
- net 3V3A: now also C1215.1
- net 3V3D: now also C1213.1; no longer C1215.1
- net 5VMAIN: now also C1211.1, C1210.1; no longer C1212.1, C1213.1
- net FT3V3: now also C1209.1; no longer C1211.1
- net GND: now also C1209.2, C1210.2
- net VBUS_CLEAN: no longer C1206.1
- net at D1201.1 (K), F1201.2, FB1201.2: now also C1201.1
Other:
- moved on the sheet: C1201
