File: ref_in.kicad_sch (KiCad schematic)
At the start: 16 parts, among them U1101 74LVC2GU04, U1102 74LVC2G04

Commit message: Fix: correct BAT54 PN and package - SOD323 not SOD323F
Parts:
- D1102, D1103: value BAT54J -> BAT54HGW; footprint Diode_SMD:D_SOD-323F -> Diode_SMD:D_SOD-323
Changed lines of the file:
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@@
       (effects (font (size 1.27 1.27)) (justify left))
     )
-    (property "Value" "BAT54J" (id 1) (at 132.842 97.9047 90)
-      (effects (font (size 1.27 1.27)) (justify left))
-    )
-    (property "Footprint" "Diode_SMD:D_SOD-323F" (id 2) (at 126.365 96.52 0)
+    (property "Value" "BAT54HGW" (id 1) (at 132.842 97.9047 90)
+      (effects (font (size 1.27 1.27)) (justify left))
+    )
+    (property "Footprint" "Diode_SMD:D_SOD-323" (id 2) (at 126.365 96.52 0)
       (effects (font (size 1.27 1.27)) hide)
     )
@@
       (effects (font (size 1.27 1.27)) (justify left))
     )
-    (property "Value" "BAT54J" (id 1) (at 131.572 108.0647 90)
-      (effects (font (size 1.27 1.27)) (justify left))
-    )
-    (property "Footprint" "Diode_SMD:D_SOD-323F" (id 2) (at 125.095 106.68 0)
-      (effects (font (size 1.27 1.27)) hide)
-    )
+    (property "Value" "BAT54HGW" (id 1) (at 131.572 108.0647 90)
+      (effects (font (size 1.27 1.27)) (justify left))
+    )
+    (property "Footprint" "Diode_SMD:D_SOD-323" (id 2) (at 125.095 106.68 0)
+      (effects (font (size 1.27 1.27)) hide)
+    )
